File: pcb/Gnarboard/Gnarboard.kicad_pcb (KiCad board)
At the start: 2 copper layers, 2 parts, among them U2 MCP3208

Commit message: a bit more progress on the design. kicad pretty decent these days.
Parts:
- added C1: 100nF, Capacitor_THT:C_Disc_D4.7mm_W2.5mm_P5.00mm, F.Cu at (83.9, 106.7)
- added C2: 100uF, Capacitor_THT:CP_Radial_D8.0mm_P5.00mm, F.Cu at (83.9, 116.8)
- added D1: 30V, Diode_THT:D_DO-35_SOD27_P10.16mm_Horizontal, F.Cu at (81.3, 76.2)
- added U3: ~, gnarboard:DF1768, F.Cu at (86.4, 91.4)
Connections:
- U1 pad 14: unconnected-(U1-GND-Pad14) -> GNDD
- U1 pad 19: +5V -> unconnected-(U1-5V0-Pad19)
- U1 pad 29: unconnected-(U1-GPIO5-Pad29) -> Net-(U1-GPIO5)
- U1 pad 30: unconnected-(U1-GPIO18-Pad30) -> Net-(U1-GPIO18)
- U1 pad 31: unconnected-(U1-GPIO19-Pad31) -> Net-(U1-GPIO19)
- U1 pad 32: unconnected-(U1-GND-Pad32) -> GNDD
- U1 pad 37: unconnected-(U1-GPIO23-Pad37) -> Net-(U1-GPIO23)
- U1 pad 38: unconnected-(U1-GND-Pad38) -> GNDD
- U2 pad 10: unconnected-(U2-~{CS}/SHDN-Pad10) -> Net-(U1-GPIO5)
- U2 pad 11: unconnected-(U2-Din-Pad11) -> Net-(U1-GPIO23)
- U2 pad 12: unconnected-(U2-Dout-Pad12) -> Net-(U1-GPIO19)
- U2 pad 13: unconnected-(U2-CLK-Pad13) -> Net-(U1-GPIO18)
- U2 pad 14: unconnected-(U2-AGND-Pad14) -> GNDA
- U2 pad 9: unconnected-(U2-DGND-Pad9) -> GNDD

Commit message: added pololu regulator. loving kicad.
Parts:
- added U4: D24V5F3, gnarboard:D24V5FX, F.Cu at (88.9, 91.4)

Commit message: much progresso en schematico
Parts:
- added C3: 1nF, Capacitor_SMD:C_0805_2012Metric_Pad1.18x1.45mm_HandSolder, F.Cu at (166.4, 95.2)
- added C4: 4.7nF, Capacitor_SMD:C_0805_2012Metric_Pad1.18x1.45mm_HandSolder, F.Cu at (168.9, 95.2)
- added C5: 100nF, Capacitor_SMD:C_0805_2012Metric_Pad1.18x1.45mm_HandSolder, F.Cu at (171.4, 95.2)
- added D2: LED, LED_SMD:LED_0805_2012Metric_Pad1.15x1.40mm_HandSolder, F.Cu at (154.7, 85.6)
- added F1: 25A, gnarboard:ATC Bypass Fuse, F.Cu at (174.5, 85.6)
- added J1: Screw_Terminal_01x08, Connector_Phoenix_GMSTB:PhoenixContact_GMSTBVA_2,5_8-G_1x08_P7.50mm_Vertical, F.Cu at (127.6, 139.7)
- added J2: Screw_Terminal_01x08, Connector_Phoenix_GMSTB:PhoenixContact_GMSTBVA_2,5_8-G_1x08_P7.50mm_Vertical, F.Cu at (188.6, 139.7)
- added J3: Screw_Terminal_01x08, Connector_Phoenix_GMSTB:PhoenixContact_GMSTBVA_2,5_8-G_1x08_P7.50mm_Vertical, F.Cu at (160.9, 38.8)
- added J4: Screw_Terminal_01x08, Connector_Phoenix_GMSTB:PhoenixContact_GMSTBVA_2,5_8-G_1x08_P7.50mm_Vertical, F.Cu at (178.4, 154.9)
- added Q1: IRF4905, Package_TO_SOT_SMD:TO-263-2, F.Cu at (171.1, 71.4)
- added Q2: MMBT5551L, Package_TO_SOT_SMD:SOT-23, F.Cu at (150.6, 66.8)
- added R1: 10k, Resistor_SMD:R_0805_2012Metric_Pad1.20x1.40mm_HandSolder, F.Cu at (155.7, 72.9)
- added R2: 1k, Resistor_SMD:R_0805_2012Metric_Pad1.20x1.40mm_HandSolder, F.Cu at (155.7, 75.8)
- added R3: 100k, Resistor_SMD:R_0805_2012Metric_Pad1.20x1.40mm_HandSolder, F.Cu at (155.7, 78.8)
- added R4: 10k, Resistor_SMD:R_0805_2012Metric_Pad1.20x1.40mm_HandSolder, F.Cu at (155.7, 81.7)
- added U5: ACS725xLCTR-20AU, Package_SO:SOIC-8_3.9x4.9mm_P1.27mm, F.Cu at (158.9, 94.3)
- C1: footprint Capacitor_THT:C_Disc_D4.7mm_W2.5mm_P5.00mm -> Capacitor_SMD:C_0805_2012Metric_Pad1.18x1.45mm_HandSolder
- U2: footprint Package_DIP:DIP-16_W7.62mm -> Package_SO:SOIC-16_3.9x9.9mm_P1.27mm
- moved U2 8.52 mm to (146.1, 96.5), turned to 180 degrees
Connections:
- U1 pad 10: unconnected-(U1-GPIO26-Pad10) -> PWM3
- U1 pad 11: unconnected-(U1-GPIO27-Pad11) -> PWM4
- U1 pad 12: unconnected-(U1-GPIO14-Pad12) -> PWM5
- U1 pad 13: unconnected-(U1-GPIO12-Pad13) -> PWM6
- U1 pad 15: unconnected-(U1-GPIO13-Pad15) -> PWM7
- U1 pad 7: unconnected-(U1-GPIO32-Pad7) -> PWM0
- U1 pad 8: unconnected-(U1-GPIO33-Pad8) -> PWM1
- U1 pad 9: unconnected-(U1-GPIO25-Pad9) -> PWM2
- U2 pad 1: unconnected-(U2-CH0-Pad1) -> ADC0
- U2 pad 2: unconnected-(U2-CH1-Pad2) -> ADC1
- U2 pad 3: unconnected-(U2-CH2-Pad3) -> ADC2
- U2 pad 4: unconnected-(U2-CH3-Pad4) -> ADC3
- U2 pad 5: unconnected-(U2-CH4-Pad5) -> ADC4
- U2 pad 6: unconnected-(U2-CH5-Pad6) -> ADC5
- U2 pad 7: unconnected-(U2-CH6-Pad7) -> ADC6
- U2 pad 8: unconnected-(U2-CH7-Pad8) -> ADC7

Commit message: wow, kicad hierarchical sheets... epic.
Parts:
- added C10: 100nF, Capacitor_SMD:C_0805_2012Metric_Pad1.18x1.45mm_HandSolder, F.Cu at (195.0, 70.2)
- added C11: 4.7nF, Capacitor_SMD:C_0805_2012Metric_Pad1.18x1.45mm_HandSolder, F.Cu at (195.0, 73.2)
- added C12: 1nF, Capacitor_SMD:C_0805_2012Metric_Pad1.18x1.45mm_HandSolder, F.Cu at (133.7, 103.0)
- added C13: 100nF, Capacitor_SMD:C_0805_2012Metric_Pad1.18x1.45mm_HandSolder, F.Cu at (133.7, 106.0)
- added C14: 4.7nF, Capacitor_SMD:C_0805_2012Metric_Pad1.18x1.45mm_HandSolder, F.Cu at (133.7, 109.0)
- added C15: 1nF, Capacitor_SMD:C_0805_2012Metric_Pad1.18x1.45mm_HandSolder, F.Cu at (133.7, 132.5)
- added C16: 100nF, Capacitor_SMD:C_0805_2012Metric_Pad1.18x1.45mm_HandSolder, F.Cu at (133.7, 135.5)
- added C17: 4.7nF, Capacitor_SMD:C_0805_2012Metric_Pad1.18x1.45mm_HandSolder, F.Cu at (133.7, 138.5)
- added C18: 1nF, Capacitor_SMD:C_0805_2012Metric_Pad1.18x1.45mm_HandSolder, F.Cu at (101.4, 103.0)
- added C19: 100nF, Capacitor_SMD:C_0805_2012Metric_Pad1.18x1.45mm_HandSolder, F.Cu at (101.4, 106.0)
- added C20: 4.7nF, Capacitor_SMD:C_0805_2012Metric_Pad1.18x1.45mm_HandSolder, F.Cu at (101.4, 109.0)
- added C21: 1nF, Capacitor_SMD:C_0805_2012Metric_Pad1.18x1.45mm_HandSolder, F.Cu at (101.4, 132.5)
- added C22: 100nF, Capacitor_SMD:C_0805_2012Metric_Pad1.18x1.45mm_HandSolder, F.Cu at (101.4, 135.5)
- added C23: 4.7nF, Capacitor_SMD:C_0805_2012Metric_Pad1.18x1.45mm_HandSolder, F.Cu at (101.4, 138.5)
- added C24: 1nF, Capacitor_SMD:C_0805_2012Metric_Pad1.18x1.45mm_HandSolder, F.Cu at (166.0, 103.0)
- added C25: 100nF, Capacitor_SMD:C_0805_2012Metric_Pad1.18x1.45mm_HandSolder, F.Cu at (166.0, 106.0)
- added C26: 4.7nF, Capacitor_SMD:C_0805_2012Metric_Pad1.18x1.45mm_HandSolder, F.Cu at (166.0, 109.0)
- added C6: 1nF, Capacitor_SMD:C_0805_2012Metric_Pad1.18x1.45mm_HandSolder, F.Cu at (166.0, 132.5)
- added C7: 100nF, Capacitor_SMD:C_0805_2012Metric_Pad1.18x1.45mm_HandSolder, F.Cu at (166.0, 135.5)
- added C8: 4.7nF, Capacitor_SMD:C_0805_2012Metric_Pad1.18x1.45mm_HandSolder, F.Cu at (166.0, 138.5)
- added C9: 1nF, Capacitor_SMD:C_0805_2012Metric_Pad1.18x1.45mm_HandSolder, F.Cu at (195.0, 67.2)
- added D3: LED, LED_SMD:LED_0805_2012Metric_Pad1.15x1.40mm_HandSolder, F.Cu at (166.1, 141.6)
- added D4: LED, LED_SMD:LED_0805_2012Metric_Pad1.15x1.40mm_HandSolder, F.Cu at (195.0, 76.2)
- added D5: LED, LED_SMD:LED_0805_2012Metric_Pad1.15x1.40mm_HandSolder, F.Cu at (133.7, 112.0)
- added D6: LED, LED_SMD:LED_0805_2012Metric_Pad1.15x1.40mm_HandSolder, F.Cu at (133.7, 141.6)
- added D7: LED, LED_SMD:LED_0805_2012Metric_Pad1.15x1.40mm_HandSolder, F.Cu at (101.4, 112.0)
- added D8: LED, LED_SMD:LED_0805_2012Metric_Pad1.15x1.40mm_HandSolder, F.Cu at (101.4, 141.6)
- added D9: LED, LED_SMD:LED_0805_2012Metric_Pad1.15x1.40mm_HandSolder, F.Cu at (166.1, 112.0)
- added F2: 25A, gnarboard:ATC Bypass Fuse, F.Cu at (155.7, 126.7)
- added F3: 25A, gnarboard:ATC Bypass Fuse, F.Cu at (184.7, 61.3)
- added F4: 25A, gnarboard:ATC Bypass Fuse, F.Cu at (123.4, 97.1)
- added F5: 25A, gnarboard:ATC Bypass Fuse, F.Cu at (123.4, 126.7)
- added F6: 25A, gnarboard:ATC Bypass Fuse, F.Cu at (91.1, 97.1)
- added F7: 25A, gnarboard:ATC Bypass Fuse, F.Cu at (91.1, 126.7)
- added F8: 25A, gnarboard:ATC Bypass Fuse, F.Cu at (155.7, 97.1)
- added Q10: IRF4905, Package_TO_SOT_SMD:TO-263-2, F.Cu at (119.6, 137.2)
- added Q11: MMBT5551L, Package_TO_SOT_SMD:SOT-23, F.Cu at (87.5, 116.1)
- added Q12: IRF4905, Package_TO_SOT_SMD:TO-263-2, F.Cu at (87.3, 107.7)
- added Q13: MMBT5551L, Package_TO_SOT_SMD:SOT-23, F.Cu at (87.5, 145.6)
- added Q14: IRF4905, Package_TO_SOT_SMD:TO-263-2, F.Cu at (87.3, 137.2)
- added Q15: MMBT5551L, Package_TO_SOT_SMD:SOT-23, F.Cu at (152.1, 116.1)
- added Q16: IRF4905, Package_TO_SOT_SMD:TO-263-2, F.Cu at (151.9, 107.7)
- added Q3: MMBT5551L, Package_TO_SOT_SMD:SOT-23, F.Cu at (152.1, 145.6)
- added Q4: IRF4905, Package_TO_SOT_SMD:TO-263-2, F.Cu at (151.9, 137.2)
- added Q5: MMBT5551L, Package_TO_SOT_SMD:SOT-23, F.Cu at (181.0, 80.2)
- added Q6: IRF4905, Package_TO_SOT_SMD:TO-263-2, F.Cu at (180.9, 71.8)
- added Q7: MMBT5551L, Package_TO_SOT_SMD:SOT-23, F.Cu at (119.8, 116.1)
- added Q8: IRF4905, Package_TO_SOT_SMD:TO-263-2, F.Cu at (119.6, 107.7)
- added Q9: MMBT5551L, Package_TO_SOT_SMD:SOT-23, F.Cu at (119.8, 145.6)
- added R10: 10k, Resistor_SMD:R_0805_2012Metric_Pad1.20x1.40mm_HandSolder, F.Cu at (190.2, 70.1)
- added R11: 10k, Resistor_SMD:R_0805_2012Metric_Pad1.20x1.40mm_HandSolder, F.Cu at (190.2, 73.0)
- added R12: 100k, Resistor_SMD:R_0805_2012Metric_Pad1.20x1.40mm_HandSolder, F.Cu at (190.2, 76.0)
- added R13: 1k, Resistor_SMD:R_0805_2012Metric_Pad1.20x1.40mm_HandSolder, F.Cu at (128.9, 103.0)
- added R14: 10k, Resistor_SMD:R_0805_2012Metric_Pad1.20x1.40mm_HandSolder, F.Cu at (128.9, 105.9)
- added R15: 10k, Resistor_SMD:R_0805_2012Metric_Pad1.20x1.40mm_HandSolder, F.Cu at (128.9, 108.9)
- added R16: 100k, Resistor_SMD:R_0805_2012Metric_Pad1.20x1.40mm_HandSolder, F.Cu at (128.9, 111.8)
- added R17: 1k, Resistor_SMD:R_0805_2012Metric_Pad1.20x1.40mm_HandSolder, F.Cu at (128.9, 132.5)
- added R18: 10k, Resistor_SMD:R_0805_2012Metric_Pad1.20x1.40mm_HandSolder, F.Cu at (128.9, 135.4)
- added R19: 10k, Resistor_SMD:R_0805_2012Metric_Pad1.20x1.40mm_HandSolder, F.Cu at (128.9, 138.4)
- added R20: 100k, Resistor_SMD:R_0805_2012Metric_Pad1.20x1.40mm_HandSolder, F.Cu at (128.9, 141.3)
- added R21: 1k, Resistor_SMD:R_0805_2012Metric_Pad1.20x1.40mm_HandSolder, F.Cu at (96.6, 103.0)
- added R22: 10k, Resistor_SMD:R_0805_2012Metric_Pad1.20x1.40mm_HandSolder, F.Cu at (96.6, 105.9)
- added R23: 10k, Resistor_SMD:R_0805_2012Metric_Pad1.20x1.40mm_HandSolder, F.Cu at (96.6, 108.9)
- added R24: 100k, Resistor_SMD:R_0805_2012Metric_Pad1.20x1.40mm_HandSolder, F.Cu at (96.6, 111.8)
- added R25: 1k, Resistor_SMD:R_0805_2012Metric_Pad1.20x1.40mm_HandSolder, F.Cu at (96.6, 132.5)
- added R26: 10k, Resistor_SMD:R_0805_2012Metric_Pad1.20x1.40mm_HandSolder, F.Cu at (96.6, 135.4)
- added R27: 10k, Resistor_SMD:R_0805_2012Metric_Pad1.20x1.40mm_HandSolder, F.Cu at (96.6, 138.4)
- added R28: 100k, Resistor_SMD:R_0805_2012Metric_Pad1.20x1.40mm_HandSolder, F.Cu at (96.6, 141.3)
- added R29: 1k, Resistor_SMD:R_0805_2012Metric_Pad1.20x1.40mm_HandSolder, F.Cu at (161.3, 103.0)
- added R30: 10k, Resistor_SMD:R_0805_2012Metric_Pad1.20x1.40mm_HandSolder, F.Cu at (161.3, 105.9)
- added R31: 10k, Resistor_SMD:R_0805_2012Metric_Pad1.20x1.40mm_HandSolder, F.Cu at (161.3, 108.9)
- added R32: 100k, Resistor_SMD:R_0805_2012Metric_Pad1.20x1.40mm_HandSolder, F.Cu at (161.3, 111.8)
- added R5: 1k, Resistor_SMD:R_0805_2012Metric_Pad1.20x1.40mm_HandSolder, F.Cu at (161.3, 132.5)
- added R6: 10k, Resistor_SMD:R_0805_2012Metric_Pad1.20x1.40mm_HandSolder, F.Cu at (161.3, 135.4)
- added R7: 10k, Resistor_SMD:R_0805_2012Metric_Pad1.20x1.40mm_HandSolder, F.Cu at (161.3, 138.4)
- added R8: 100k, Resistor_SMD:R_0805_2012Metric_Pad1.20x1.40mm_HandSolder, F.Cu at (161.3, 141.3)
- added R9: 1k, Resistor_SMD:R_0805_2012Metric_Pad1.20x1.40mm_HandSolder, F.Cu at (190.2, 67.1)
- added U10: ACS725xLCTR-20AU, Package_SO:SOIC-8_3.9x4.9mm_P1.27mm, F.Cu at (80.8, 117.1)
- added U11: ACS725xLCTR-20AU, Package_SO:SOIC-8_3.9x4.9mm_P1.27mm, F.Cu at (80.8, 146.6)
- added U12: ACS725xLCTR-20AU, Package_SO:SOIC-8_3.9x4.9mm_P1.27mm, F.Cu at (145.4, 117.1)
- added U6: ACS725xLCTR-20AU, Package_SO:SOIC-8_3.9x4.9mm_P1.27mm, F.Cu at (145.4, 146.6)
- added U7: ACS725xLCTR-20AU, Package_SO:SOIC-8_3.9x4.9mm_P1.27mm, F.Cu at (174.4, 81.2)
- added U8: ACS725xLCTR-20AU, Package_SO:SOIC-8_3.9x4.9mm_P1.27mm, F.Cu at (113.1, 117.1)
- added U9: ACS725xLCTR-20AU, Package_SO:SOIC-8_3.9x4.9mm_P1.27mm, F.Cu at (113.1, 146.6)
- C4: value 4.7nF -> 100nF
- C5: value 100nF -> 4.7nF
- Q1: value IRF4905 -> MMBT5551L; footprint Package_TO_SOT_SMD:TO-263-2 -> Package_TO_SOT_SMD:SOT-23
- Q2: value MMBT5551L -> IRF4905; footprint Package_TO_SOT_SMD:SOT-23 -> Package_TO_SOT_SMD:TO-263-2
- R1: value 10k -> 1k
- R2: value 1k -> 10k
- R3: value 100k -> 10k
- R4: value 10k -> 100k
- moved J2 122.7 mm to (110.9, 44.8)
- moved J4 110.9 mm to (110.9, 67.0)
- moved J1 107.3 mm to (110.9, 33.7)
- moved C2 83.8 mm to (157.4, 76.6)
- moved C3 64.3 mm to (195.0, 37.6), turned to 0 degrees
- moved C1 62.5 mm to (143.5, 88.1)
- moved D1 62.0 mm to (142.7, 84.8)
- moved U4 62.0 mm to (149.3, 77.4)
- moved C4 60.5 mm to (195.0, 40.6), turned to 0 degrees
- moved C5 56.7 mm to (195.0, 43.7), turned to 0 degrees
- moved D2 56.0 mm to (195.0, 46.7)
- moved F1 54.7 mm to (184.7, 31.8)
- moved U1 53.4 mm to (78.6, 35.0)
- moved J3 52.8 mm to (110.9, 55.9)
- moved R1 49.3 mm to (190.2, 37.6)
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Connections:
- C4 pad 1: ADC0 -> +3.3V
- C5 pad 1: +3.3V -> /CHANNEL 0/ADC
- F1 pad 1: Net-(Q1-S) -> Net-(Q2-S)
- F1 pad 3: CH0+ -> /CHANNEL 0/LOAD+
- J1 pad 1: CH0+ -> /CHANNEL 0/LOAD-
- J1 pad 2: CH0- -> /CHANNEL 0/LOAD+
- J1 pad 3: CH1+ -> /CHANNEL 1/LOAD-
- J1 pad 4: CH1- -> /CHANNEL 1/LOAD+
- J1 pad 5: CH2+ -> /CHANNEL 2/LOAD-
- J1 pad 6: CH2- -> /CHANNEL 2/LOAD+
- J1 pad 7: CH3+ -> /CHANNEL 3/LOAD-
- J1 pad 8: CH3- -> /CHANNEL 3/LOAD+
- J2 pad 1: CH4+ -> /CHANNEL 4/LOAD-
- J2 pad 2: CH4- -> /CHANNEL 4/LOAD+
- J2 pad 3: CH5+ -> /CHANNEL 5/LOAD-
- J2 pad 4: CH5- -> /CHANNEL 5/LOAD+
- J2 pad 5: CH6+ -> /CHANNEL 6/LOAD-
- J2 pad 6: CH6- -> /CHANNEL 6/LOAD+
- J2 pad 7: CH7+ -> /CHANNEL 7/LOAD-
- J2 pad 8: CH7- -> /CHANNEL 7/LOAD+
- Q1 pad 1: Net-(Q1-G) -> Net-(Q1-B)
- Q1 pad 2: CH0+ -> GNDD
- Q1 pad 3: Net-(Q1-S) -> Net-(Q1-C)
- Q2 pad 1: Net-(Q2-B) -> Net-(Q2-G)
- Q2 pad 2: GNDD -> /CHANNEL 0/LOAD+
- Q2 pad 3: Net-(Q2-C) -> Net-(Q2-S)
- R1 pad 1: PWM0 -> Net-(D2-A)
- R1 pad 2: Net-(Q2-B) -> /CHANNEL 0/PWM
- R2 pad 1: Net-(D2-A) -> /CHANNEL 0/PWM
- R2 pad 2: PWM0 -> Net-(Q1-B)
- R3 pad 1: Net-(Q2-C) -> Net-(Q2-G)
- R3 pad 2: Net-(Q1-G) -> +24V
- R4 pad 1: Net-(Q1-G) -> Net-(Q1-C)
- R4 pad 2: +24V -> Net-(Q2-G)
- U1 pad 10: PWM3 -> /CHANNEL 3/PWM
- U1 pad 11: PWM4 -> /CHANNEL 4/PWM
- U1 pad 12: PWM5 -> /CHANNEL 5/PWM
- U1 pad 13: PWM6 -> /CHANNEL 6/PWM
- U1 pad 15: PWM7 -> /CHANNEL 7/PWM
- U1 pad 7: PWM0 -> /CHANNEL 0/PWM
- U1 pad 8: PWM1 -> /CHANNEL 1/PWM
- U1 pad 9: PWM2 -> /CHANNEL 2/PWM
- U2 pad 1: ADC0 -> /CHANNEL 0/ADC
- U2 pad 2: ADC1 -> /CHANNEL 1/ADC
- U2 pad 3: ADC2 -> /CHANNEL 2/ADC
- U2 pad 4: ADC3 -> /CHANNEL 3/ADC
- U2 pad 5: ADC4 -> /CHANNEL 4/ADC
- U2 pad 6: ADC5 -> /CHANNEL 5/ADC
- U2 pad 7: ADC6 -> /CHANNEL 6/ADC
- U2 pad 8: ADC7 -> /CHANNEL 7/ADC
- U5 pad 1: CH0- -> /CHANNEL 0/LOAD-
- U5 pad 2: CH0- -> /CHANNEL 0/LOAD-
- U5 pad 7: ADC0 -> /CHANNEL 0/ADC

Commit message: big kicad progress.
Parts:
- removed C2: 100uF, Capacitor_THT:CP_Radial_D8.0mm_P5.00mm
- J3, J4: value Screw_Terminal_01x08 -> Screw_Terminal_01x12; footprint Connector_Phoenix_GMSTB:PhoenixContact_GMSTBVA_2,5_8-G_1x08_P7.50mm_Vertical -> gnarboard:BSS 2301
- moved D3 423.3 mm to (-252.5, 78.5), turned to -90 degrees
- moved C8 419.8 mm to (-249.5, 78.5), turned to -90 degrees
- moved R8 419.0 mm to (-252.3, 73.7), turned to -90 degrees
- moved Q3 416.6 mm to (-256.5, 64.6), turned to -90 degrees
- moved C7 416.4 mm to (-246.5, 78.5), turned to -90 degrees
- moved R7 415.6 mm to (-249.3, 73.7), turned to -90 degrees
- moved C6 413.0 mm to (-243.5, 78.5), turned to -90 degrees
- moved U6 412.6 mm to (-257.5, 57.9), turned to -90 degrees
- moved R6 412.3 mm to (-246.4, 73.7), turned to -90 degrees
- moved R5 408.9 mm to (-243.4, 73.7), turned to -90 degrees
- moved D6 397.8 mm to (-252.5, 46.2), turned to -90 degrees
- moved F2 397.6 mm to (-237.6, 68.2), turned to -90 degrees
- moved C17 394.2 mm to (-249.5, 46.2), turned to -90 degrees
- moved R20 394.1 mm to (-252.3, 41.4), turned to -90 degrees
- moved Q9 393.0 mm to (-256.5, 32.3), turned to -90 degrees
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Connections:
- net /CHANNEL 0/ADC renamed /ADC0
- net /CHANNEL 0/PWM renamed /PWM0
- net /CHANNEL 1/ADC renamed /ADC1
- net /CHANNEL 1/PWM renamed /PWM1
- net /CHANNEL 2/ADC renamed /ADC2
- net /CHANNEL 2/PWM renamed /PWM2
- net /CHANNEL 3/ADC renamed /ADC3
- net /CHANNEL 3/PWM renamed /PWM3
- net /CHANNEL 4/ADC renamed /ADC4
- net /CHANNEL 4/PWM renamed /PWM4
- net /CHANNEL 5/ADC renamed /ADC5
- net /CHANNEL 5/PWM renamed /PWM5
- net /CHANNEL 6/ADC renamed /ADC6
- net /CHANNEL 6/PWM renamed /PWM6
- net /CHANNEL 7/ADC renamed /ADC7
- net /CHANNEL 7/PWM renamed /PWM7
- F1 pad 3: /CHANNEL 0/LOAD+ -> /CH+0
- F2 pad 3: /CHANNEL 1/LOAD+ -> /CH+1
- F3 pad 3: /CHANNEL 2/LOAD+ -> /CH+2
- F4 pad 3: /CHANNEL 3/LOAD+ -> /CH+3
- F5 pad 3: /CHANNEL 4/LOAD+ -> /CH+4
- F6 pad 3: /CHANNEL 5/LOAD+ -> /CH+5
- F7 pad 3: /CHANNEL 6/LOAD+ -> /CH+6
- F8 pad 3: /CHANNEL 7/LOAD+ -> /CH+7
- J1 pad 1: /CHANNEL 0/LOAD- -> /CH+0
- J1 pad 2: /CHANNEL 0/LOAD+ -> /CH-0
- J1 pad 3: /CHANNEL 1/LOAD- -> /CH+1
- J1 pad 4: /CHANNEL 1/LOAD+ -> /CH-1
- J1 pad 5: /CHANNEL 2/LOAD- -> /CH+2
- J1 pad 6: /CHANNEL 2/LOAD+ -> /CH-2
- J1 pad 7: /CHANNEL 3/LOAD- -> /CH+3
- J1 pad 8: /CHANNEL 3/LOAD+ -> /CH-3
- J2 pad 1: /CHANNEL 4/LOAD- -> /CH+4
- J2 pad 2: /CHANNEL 4/LOAD+ -> /CH-4
- J2 pad 3: /CHANNEL 5/LOAD- -> /CH+5
- J2 pad 4: /CHANNEL 5/LOAD+ -> /CH-5
- J2 pad 5: /CHANNEL 6/LOAD- -> /CH+6
- J2 pad 6: /CHANNEL 6/LOAD+ -> /CH-6
- J2 pad 7: /CHANNEL 7/LOAD- -> /CH+7
- J2 pad 8: /CHANNEL 7/LOAD+ -> /CH-7
- Q10 pad 2: /CHANNEL 4/LOAD+ -> /CH+4
- Q12 pad 2: /CHANNEL 5/LOAD+ -> /CH+5
- Q14 pad 2: /CHANNEL 6/LOAD+ -> /CH+6
- Q16 pad 2: /CHANNEL 7/LOAD+ -> /CH+7
- Q2 pad 2: /CHANNEL 0/LOAD+ -> /CH+0
- Q4 pad 2: /CHANNEL 1/LOAD+ -> /CH+1
- Q6 pad 2: /CHANNEL 2/LOAD+ -> /CH+2
- Q8 pad 2: /CHANNEL 3/LOAD+ -> /CH+3
- U10 pad 1: /CHANNEL 5/LOAD- -> /CH-5
- U10 pad 2: /CHANNEL 5/LOAD- -> /CH-5
- U11 pad 1: /CHANNEL 6/LOAD- -> /CH-6
- U11 pad 2: /CHANNEL 6/LOAD- -> /CH-6
- U12 pad 1: /CHANNEL 7/LOAD- -> /CH-7
- U12 pad 2: /CHANNEL 7/LOAD- -> /CH-7
- U5 pad 1: /CHANNEL 0/LOAD- -> /CH-0
- U5 pad 2: /CHANNEL 0/LOAD- -> /CH-0
- U6 pad 1: /CHANNEL 1/LOAD- -> /CH-1
- U6 pad 2: /CHANNEL 1/LOAD- -> /CH-1
- U7 pad 1: /CHANNEL 2/LOAD- -> /CH-2
- U7 pad 2: /CHANNEL 2/LOAD- -> /CH-2
- U8 pad 1: /CHANNEL 3/LOAD- -> /CH-3
- U8 pad 2: /CHANNEL 3/LOAD- -> /CH-3
- U9 pad 1: /CHANNEL 4/LOAD- -> /CH-4
- U9 pad 2: /CHANNEL 4/LOAD- -> /CH-4
Routing:
- net /CH+0: track 0.00 -> 72.2 mm
- net +24V: track 0.00 -> 72.0 mm
- net Net-(Q2-S): track 0.00 -> 29.2 mm
- net GNDPWR: track 0.00 -> 18.5 mm
- net GNDA: track 0.00 -> 14.6 mm
- net /CH-0: track 0.00 -> 14.1 mm
- net Net-(Q2-G): track 0.00 -> 9.18 mm
- net Net-(D2-A): track 0.00 -> 7.39 mm
- net Net-(U5-FILTER): track 0.00 -> 5.90 mm
- net +3.3V: track 0.00 -> 5.90 mm
- net /ADC0: track 0.00 -> 5.38 mm
- net /PWM0: track 0.00 -> 4.32 mm
- net Net-(Q1-C): track 0.00 -> 3.65 mm
- net GNDD: track 0.00 -> 3.36 mm
- net Net-(Q1-B): track 0.00 -> 2.63 mm
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
Commit message: layout and outline starting to look pretty good.
Parts:
- moved U11 465.6 mm to (187.8, 129.3), turned to 0 degrees
- moved C23 459.9 mm to (195.8, 128.7), turned to 0 degrees
- moved Q13 457.0 mm to (191.9, 87.8), turned to 180 degrees
- moved C22 456.3 mm to (195.8, 126.1), turned to 0 degrees
- moved C21 454.7 mm to (195.8, 131.2), turned to 0 degrees
- moved R28 451.7 mm to (191.9, 91.2), turned to 0 degrees
- moved D8 450.0 mm to (191.9, 84.8), turned to 180 degrees
- moved R27 449.3 mm to (191.9, 93.7), turned to 180 degrees
- moved R26 443.9 mm to (191.9, 79.8), turned to 0 degrees
- moved R25 441.4 mm to (191.9, 82.3), turned to 0 degrees
- moved U12 436.7 mm to (202.8, 129.3), turned to 0 degrees
- moved Q15 434.5 mm to (206.9, 87.8), turned to 180 degrees
- moved C26 433.7 mm to (210.8, 128.7), turned to 0 degrees
- moved F7 433.3 mm to (191.4, 64.8), turned to 90 degrees
- moved C25 430.4 mm to (210.8, 126.1), turned to 0 degrees
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Routing:
- net /CH+3: track 0.00 -> 76.6 mm
- net /CH+7: track 0.00 -> 76.6 mm
- net /CH+6: track 0.00 -> 76.6 mm
- net /CH+5: track 0.00 -> 76.6 mm
- net /CH+4: track 0.00 -> 76.6 mm
- net /CH+2: track 0.00 -> 76.6 mm
- net /CH+1: track 0.00 -> 76.6 mm
- net GNDA: track 14.6 -> 58.1 mm, vias 0 -> 1
- net +3.3V: track 5.90 -> 40.3 mm, vias 0 -> 8
- net GNDD: track 3.36 -> 34.0 mm, vias 0 -> 8
- net Net-(Q8-S): track 0.00 -> 29.3 mm
- net Net-(Q14-S): track 0.00 -> 29.3 mm
- net Net-(Q12-S): track 0.00 -> 29.3 mm
- net Net-(Q10-S): track 0.00 -> 29.3 mm
- net Net-(Q16-S): track 0.00 -> 29.3 mm
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Other:
- board outline added: 157.5 x 124.5 mm

Commit message: board mostly laid out.
Parts:
- added JP1: SolderJumper_2_Bridged, Jumper:SolderJumper-2_P1.3mm_Bridged_RoundedPad1.0x1.5mm, F.Cu at (81.8, 121.7)
- added JP2: SolderJumper_2_Bridged, Jumper:SolderJumper-2_P1.3mm_Bridged_RoundedPad1.0x1.5mm, F.Cu at (81.8, 136.1)
- D1: footprint Diode_THT:D_DO-35_SOD27_P10.16mm_Horizontal -> Diode_SMD:D_SOD-123
- moved U2 25.4 mm to (76.2, 128.3)
- moved D1 7.18 mm to (85.1, 62.2)
- moved Q10 1.25 mm to (159.5, 105.4)
- moved Q12 1.25 mm to (174.5, 105.4)
- moved Q14 1.25 mm to (189.5, 105.4)
- moved Q16 1.25 mm to (204.5, 105.4)
- moved Q4 1.25 mm to (114.5, 105.4)
- moved Q6 1.25 mm to (129.5, 105.4)
- moved Q8 1.25 mm to (144.5, 105.4)
- moved C10 1.06 mm to (134.8, 126.1)
- moved C11 1.06 mm to (134.8, 128.7)
- moved C12 1.06 mm to (149.8, 131.2)
- moved C13 1.06 mm to (149.8, 126.1)
- moved C14 1.06 mm to (149.8, 128.6)
- moved C15 1.06 mm to (164.8, 131.2)
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Connections:
- D1 pad 2: GNDPWR -> GNDD
- U3 pad 4: GNDA -> GNDD
- U3 pad 5: GNDPWR -> GNDD
- U3 pad 6: GNDPWR -> GNDD
- U4 pad 3: +24V -> GNDD
Routing:
- net +24V: track 49.9 -> 719.0 mm
- net +3.3V: track 40.3 -> 280.2 mm, vias 8 -> 9
- net /PWM7: track 4.67 -> 162.4 mm
- net /PWM6: track 4.67 -> 146.8 mm
- net /ADC7: track 4.51 -> 145.9 mm, vias 1 -> 2
- net /PWM5: track 4.67 -> 131.2 mm
- net /ADC6: track 4.51 -> 131.0 mm, vias 1 -> 2
- net /ADC5: track 4.51 -> 116.2 mm, vias 1 -> 2
- net /PWM4: track 4.67 -> 114.7 mm
- net /ADC4: track 4.51 -> 101.2 mm, vias 1 -> 2
- net /PWM3: track 4.67 -> 99.1 mm
- net /ADC3: track 4.51 -> 86.4 mm, vias 1 -> 2
- net /PWM2: track 4.67 -> 82.6 mm
- net /ADC2: track 4.51 -> 71.6 mm, vias 1 -> 2
- net /PWM1: track 4.67 -> 63.6 mm
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- added copper zone on B.Cu, net +24V
- added copper zone on F.Cu, net +24V
- added copper zone on F.Cu, net /CH-0
- added copper zone on F.Cu, net /CH-1
- added copper zone on F.Cu, net /CH-2
- added copper zone on F.Cu, net /CH-3
- added copper zone on F.Cu, net /CH-4
- added copper zone on F.Cu, net /CH-5
- added copper zone on F.Cu, net /CH-6
- added copper zone on F.Cu, net /CH-7
- added copper zone on B.Cu, net GNDA
- added copper zone on F.Cu, net GNDA
- added copper zone on B.Cu, net GNDD
- added copper zone on F.Cu, net GNDD
- added copper zone on B.Cu, net GNDPWR
- added copper zone on F.Cu, net GNDPWR
