File: pcb/Gnarboard/mosfet.kicad_sch (KiCad schematic)
At the start: 15 parts, among them J5 Screw_Terminal_01x02, Q1 IRF4905, Q2 MMBT5551L, U5 ACS725xLCTR-20AU

Commit message: went over components again, should be ready to rock and roll!
Parts:
- D10: value GS1G-LTP -> SS16; Vendor 833-GS1G-LTP -> 625-SS16-E3
- Q2: value MMBT5551L -> BC817; symbol Transistor_BJT:MMBT5551L -> Transistor_BJT:BC817; Vendor 637-MMBT5551 -> 771-BC817-25-T/R
- R3: value 6.8k -> 4.7k; Vendor 652-CR0805JW-682ELF -> 652-CR0805JW-472ELF
- R4: value 33k -> 22k; Vendor 652-CR0805JW-333ELF -> 652-CR0805JW-223ELF
Other:
- moved on the sheet: C5, D2, R2
Changed lines of the file:
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@@
   (junction (at 167.64 124.46) (diameter 0) (color 0 0 0 0)
   )
+  (junction (at 101.6 81.28) (diameter 0) (color 0 0 0 0)
+  )
   (junction (at 167.64 113.03) (diameter 0) (color 0 0 0 0)
   )
   (junction (at 148.59 86.36) (diameter 0) (color 0 0 0 0)
   )
-  (junction (at 104.14 81.28) (diameter 0) (color 0 0 0 0)
-  )
   (junction (at 114.3 96.52) (diameter 0) (color 0 0 0 0)
   )
@@
     (stroke (width 0) (type default))
   )
-  (wire (pts (xy 104.14 81.28) (xy 107.95 81.28))
-    (stroke (width 0) (type default))
-  )
   (wire (pts (xy 139.7 53.34) (xy 139.7 54.61))
     (stroke (width 0) (type default))
@@
     (stroke (width 0) (type default))
   )
-  (wire (pts (xy 161.29 102.87) (xy 161.29 106.68))
-    (stroke (width 0) (type default))
-  )
-  (wire (pts (xy 161.29 106.68) (xy 165.1 106.68))
+  (wire (pts (xy 149.86 102.87) (xy 163.83 102.87))
     (stroke (width 0) (type default))
   )
@@
     (stroke (width 0) (type default))
   )
-  (wire (pts (xy 104.14 96.52) (xy 114.3 96.52))
+  (wire (pts (xy 101.6 96.52) (xy 114.3 96.52))
     (stroke (width 0) (type default))
   )
@@
     (stroke (width 0) (type default))
   )
+  (wire (pts (xy 101.6 81.28) (xy 107.95 81.28))
+    (stroke (width 0) (type default))
+  )
   (wire (pts (xy 114.3 54.61) (xy 114.3 57.15))
     (stroke (width 0) (type default))
@@
     (stroke (width 0) (type default))
   )
-  (wire (pts (xy 170.18 106.68) (xy 176.53 106.68))
+  (wire (pts (xy 168.91 102.87) (xy 176.53 102.87))
     (stroke (width 0) (type default))
   )
@@
     (stroke (width 0) (type default))
   )
-  (wire (pts (xy 176.53 106.68) (xy 176.53 124.46))
-    (stroke (width 0) (type default))
-  )
-  (wire (pts (xy 104.14 82.55) (xy 104.14 81.28))
-    (stroke (width 0) (type default))
-  )
-  (wire (pts (xy 104.14 96.52) (xy 104.14 95.25))
+  (wire (pts (xy 176.53 102.87) (xy 176.53 124.46))
+    (stroke (width 0) (type default))
+  )
+  (wire (pts (xy 101.6 82.55) (xy 101.6 81.28))
+    (stroke (width 0) (type default))
+  )
+  (wire (pts (xy 101.6 96.52) (xy 101.6 95.25))
     (stroke (width 0) (type default))
   )
@@
     (stroke (width 0) (type default))
   )
-  (wire (pts (xy 96.52 81.28) (xy 104.14 81.28))
+  (wire (pts (xy 96.52 81.28) (xy 101.6 81.28))
     (stroke (width 0) (type default))
   )
@@
   )
   (wire (pts (xy 114.3 66.04) (xy 123.19 66.04))
-    (stroke (width 0) (type default))
-  )
-  (wire (pts (xy 161.29 102.87) (xy 149.86 102.87))
     (stroke (width 0) (type default))
   )
@@
       (effects (font (size 1.27 1.27)) (justify left))
     )
-    (property "Value" "GS1G-LTP" (at 165.1 86.36 90)
+    (property "Value" "SS16" (at 165.1 86.36 90)
       (effects (font (size 1.27 1.27)) (justify left))
     )
@@
       (effects (font (size 1.27 1.27)) hide)
     )
-    (property "Datasheet" "http://www.onsemi.com/pub_link/Collateral/MRA4003T3-D.PDF" (at 162.56 85.09 0)
+    (property "Datasheet" "" (at 162.56 85.09 0)
       (effects (font (size 1.27 1.27)) hide)
     )
@@
       (effects (font (size 1.27 1.27)) hide)
     )
-    (property "Vendor" "833-GS1G-LTP" (at 162.56 85.09 0)
+    (property "Vendor" "625-SS16-E3 " (at 162.56 85.09 0)
       (effects (font (size 1.27 1.27)) hide)
     )
@@
     )
   )
-  (symbol (lib_id "Device:R_Small_US") (at 104.14 85.09 180) (unit 1)
-    (in_bom yes) (on_board yes) (dnp no) (fields_autoplaced)
-    (property "Reference" "R2" (at 107.95 83.82 0)
+  (symbol (lib_id "Device:R_Small_US") (at 101.6 85.09 180) (unit 1)
+    (in_bom yes) (on_board yes) (dnp no) (fields_autoplaced)
+    (property "Reference" "R2" (at 105.41 83.82 0)
       (effects (font (size 1.27 1.27)) (justify right))
     )
-    (property "Value" "1k" (at 107.95 86.36 0)
+    (property "Value" "1k" (at 105.41 86.36 0)
       (effects (font (size 1.27 1.27)) (justify right))
     )
-    (property "Footprint" "Resistor_SMD:R_0805_2012Metric_Pad1.20x1.40mm_HandSolder" (at 104.14 85.09 0)
-      (effects (font (size 1.27 1.27)) hide)
-    )
-    (property "Datasheet" "~" (at 104.14 85.09 0)
-      (effects (font (size 1.27 1.27)) hide)
-    )
-    (property "Vendor" " 652-CR0805JW-102ELF " (at 104.14 85.09 0)
+    (property "Footprint" "Resistor_SMD:R_0805_2012Metric_Pad1.20x1.40mm_HandSolder" (at 101.6 85.09 0)
+      (effects (font (size 1.27 1.27)) hide)
+    )
+    (property "Datasheet" "~" (at 101.6 85.09 0)
+      (effects (font (size 1.27 1.27)) hide)
+    )
+    (property "Vendor" " 652-CR0805JW-102ELF " (at 101.6 85.09 0)
       (effects (font (size 1.27 1.27)) hide)
     )
@@
       (effects (font (size 1.27 1.27)) (justify right))
     )
-    (property "Value" "33k" (at 125.73 62.23 0)
+    (property "Value" "22k" (at 125.73 62.23 0)
       (effects (font (size 1.27 1.27)) (justify right))
     )
@@
       (effects (font (size 1.27 1.27)) hide)
     )
-    (property "Vendor" " 652-CR0805JW-333ELF " (at 123.19 60.96 0)
+    (property "Vendor" " 652-CR0805JW-223ELF " (at 123.19 60.96 0)
       (effects (font (size 1.27 1.27)) hide)
     )
@@
     )
   )
-  (symbol (lib_id "Device:LED") (at 104.14 91.44 90) (unit 1)
-    (in_bom yes) (on_board yes) (dnp no) (fields_autoplaced)
-    (property "Reference" "D2" (at 109.22 91.7575 90)
+  (symbol (lib_id "Device:LED") (at 101.6 91.44 90) (unit 1)
+    (in_bom yes) (on_board yes) (dnp no) (fields_autoplaced)
+    (property "Reference" "D2" (at 106.68 91.7575 90)
       (effects (font (size 1.27 1.27)) (justify right))
     )
-    (property "Value" "LED" (at 109.22 94.2975 90)
+    (property "Value" "LED" (at 106.68 94.2975 90)
       (effects (font (size 1.27 1.27)) (justify right))
     )
-    (property "Footprint" "LED_SMD:LED_0805_2012Metric_Pad1.15x1.40mm_HandSolder" (at 104.14 91.44 0)
-      (effects (font (size 1.27 1.27)) hide)
-    )
-    (property "Datasheet" "~" (at 104.14 91.44 0)
-      (effects (font (size 1.27 1.27)) hide)
-    )
-    (property "Vendor" "150080RS75000" (at 104.14 91.44 0)
+    (property "Footprint" "LED_SMD:LED_0805_2012Metric_Pad1.15x1.40mm_HandSolder" (at 101.6 91.44 0)
+      (effects (font (size 1.27 1.27)) hide)
+    )
+    (property "Datasheet" "~" (at 101.6 91.44 0)
+      (effects (font (size 1.27 1.27)) hide)
+    )
+    (property "Vendor" "150080RS75000" (at 101.6 91.44 0)
       (effects (font (size 1.27 1.27)) hide)
     )
@@
     )
   )
-  (symbol (lib_id "Device:C_Small") (at 167.64 106.68 90) (unit 1)
-    (in_bom yes) (on_board yes) (dnp no) (fields_autoplaced)
-    (property "Reference" "C5" (at 167.6463 100.33 90)
+  (symbol (lib_id "Device:C_Small") (at 166.37 102.87 90) (unit 1)
+    (in_bom yes) (on_board yes) (dnp no) (fields_autoplaced)
+    (property "Reference" "C5" (at 166.3763 96.52 90)
       (effects (font (size 1.27 1.27)))
     )
-    (property "Value" "100nF" (at 167.6463 102.87 90)
+    (property "Value" "100nF" (at 166.3763 99.06 90)
       (effects (font (size 1.27 1.27)))
     )
-    (property "Footprint" "Capacitor_SMD:C_0805_2012Metric_Pad1.18x1.45mm_HandSolder" (at 167.64 106.68 0)
-      (effects (font (size 1.27 1.27)) hide)
-    )
-    (property "Datasheet" "~" (at 167.64 106.68 0)
-      (effects (font (size 1.27 1.27)) hide)
-    )
-    (property "Vendor" "08053C104KAT4A" (at 167.64 106.68 0)
+    (property "Footprint" "Capacitor_SMD:C_0805_2012Metric_Pad1.18x1.45mm_HandSolder" (at 166.37 102.87 0)
+      (effects (font (size 1.27 1.27)) hide)
+    )
+    (property "Datasheet" "~" (at 166.37 102.87 0)
+      (effects (font (size 1.27 1.27)) hide)
+    )
+    (property "Vendor" "08053C104KAT4A" (at 166.37 102.87 0)
       (effects (font (size 1.27 1.27)) hide)
     )
@@
       (effects (font (size 1.27 1.27)) (justify right))
     )
-    (property "Value" "6.8k" (at 125.73 72.39 0)
+    (property "Value" "4.7k" (at 125.73 72.39 0)
       (effects (font (size 1.27 1.27)) (justify right))
     )
@@
       (effects (font (size 1.27 1.27)) hide)
     )
-    (property "Vendor" "652-CR0805JW-682ELF" (at 123.19 71.12 0)
+    (property "Vendor" "652-CR0805JW-472ELF" (at 123.19 71.12 0)
       (effects (font (size 1.27 1.27)) hide)
     )
@@
     )
   )
-  (symbol (lib_id "Transistor_BJT:MMBT5551L") (at 120.65 81.28 0) (unit 1)
-    (in_bom yes) (on_board yes) (dnp no) (fields_autoplaced)
+  (symbol (lib_id "Transistor_BJT:BC817") (at 120.65 81.28 0) (unit 1)
+    (in_bom yes) (on_board yes) (dnp no)
     (property "Reference" "Q2" (at 125.73 80.01 0)
       (effects (font (size 1.27 1.27)) (justify left))
     )
-    (property "Value" "MMBT5551L" (at 125.73 82.55 0)
+    (property "Value" "BC817" (at 125.73 82.55 0)
       (effects (font (size 1.27 1.27)) (justify left))
     )
@@
       (effects (font (size 1.27 1.27) italic) (justify left) hide)
     )
-    (property "Datasheet" "www.onsemi.com/pub/Collateral/MMBT5550LT1-D.PDF" (at 120.65 81.28 0)
+    (property "Datasheet" "https://www.onsemi.com/pub/Collateral/BC818-D.pdf" (at 120.65 81.28 0)
       (effects (font (size 1.27 1.27)) (justify left) hide)
     )
-    (property "Vendor" "637-MMBT5551" (at 120.65 81.28 0)
-      (effects (font (size 1.27 1.27)) hide)
-    )
+    (property "Vendor" "771-BC817-25-T/R" (at 120.65 81.28 0)
+      (effects (font (size 1.27 1.27)) hide)
+    )

Commit message: pcb stuff
Parts:
- J5: footprint gnarboard:Amphenol OQ02715 -> gnarboard:Molex 1x02 .375
Connections:
- net GNDPWR: now also D10.2 (A), J5.2 (Pin_2); no longer U5.3 (IP-), U5.4 (IP-)
- net at D10.1 (K), J5.1 (Pin_1): now also U5.3 (IP-), U5.4 (IP-); no longer F1.3, Q1.2 (D)
- net at U5.1 (IP+), U5.2 (IP+): now also F1.3, Q1.2 (D); no longer D10.2 (A), J5.2 (Pin_2)
Other:
- note added: "BYPASS FUSE"
- note added: "MOSFET Driver"
- note removed: "MOSFET"
- moved on the sheet: C3, C4, C5, D10, D18, D2, F1, J5, Q2, R1, R2, R3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

Commit message: lots of progress on new layout.
Parts:
- U5: footprint Package_SO:SOIC-8_3.9x4.9mm_P1.27mm -> gnarboard:ACS7XX
Changed lines of the file:
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@@
       (effects (font (size 1.27 1.27)) (justify left) hide)
     )
-    (property "Footprint" "Package_SO:SOIC-8_3.9x4.9mm_P1.27mm" (at 152.4 119.38 0)
+    (property "Footprint" "gnarboard:ACS7XX" (at 152.4 119.38 0)
       (effects (font (size 1.27 1.27) italic) (justify left) hide)
     )
