File: pcb/8ch-mosfet/8ch-mosfet.kicad_pcb (KiCad board)
At the start: 2 copper layers, 184 x 136 mm, 146 parts, among them J1 N2K, J10 Screw_Terminal_01x02, J11 Screw_Terminal_01x02, J12 Screw_Terminal_01x02, J2 I2C, J3 Screw_Terminal_01x09, J5 Screw_Terminal_01x02, J6 Screw_Terminal_01x02, J7 Screw_Terminal_01x02, J8 Screw_Terminal_01x02, J9 Screw_Terminal_01x02, M1 Fan_4pin, Q1 BC817, Q10 IRF4905, Q11 BC817, Q12 IRF4905, Q13 BC817, Q14 IRF4905, Q15 BC817, Q16 IRF4905, Q2 IRF4905, Q3 BC817, Q4 IRF4905, Q5 BC817, Q6 IRF4905, Q7 BC817, Q8 IRF4905, Q9 BC817, U1 ESP32-DEVKITC, U10 ACS725xLCTR-20AU, U11 ACS725xLCTR-20AU, U12 ACS725xLCTR-20AU, U2 MCP3208, U3 R-78B3.3-2.0, U5 ACS725xLCTR-20AU, U6 ACS725xLCTR-20AU, U7 ACS725xLCTR-20AU, U8 ACS725xLCTR-20AU, U9 ACS725xLCTR-20AU

Commit message: renaming and moving
Other:
- board text added: "8ch Mosfet Rev B"
- board text removed: "8ch Mosfet Rev A"
Changed lines of the file:
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@@
     (effects (font (size 1.75 1.75) (thickness 0.2)) (justify left bottom))
   )
-  (gr_text "8ch Mosfet Rev A" (at 8.666 131.834) (layer "F.SilkS")
+  (gr_text "8ch Mosfet Rev B" (at 8.666 131.834) (layer "F.SilkS")
     (effects (font (size 1.75 1.75) (thickness 0.2)) (justify left bottom))
   )
