File: boards/8ch-mosfet/mosfet.kicad_sch (KiCad schematic)
At the start: 15 parts, among them J5 Screw_Terminal_01x02, Q1 IRF4905, Q2 BC817, U5 ACS725xLCTR-20AU

Commit message: a couple tweaks to mosfet circuit
Parts:
- Q2: value BC817 -> 2N7002; symbol Transistor_BJT:BC817 -> Transistor_FET:2N7002
- R1: value 1k -> 220
Connections:
- net +24V: no longer D18.1 (K), R4.2
- net at F1.1, Q1.3 (S): now also D18.1 (K), R4.2
Other:
- moved on the sheet: F1
Changed lines of the file:
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@@
 (kicad_sch (version 20230121) (generator eeschema)
   (paper "A4")
-  (junction (at 165.1 71.12) (diameter 0) (color 0 0 0 0)
+  (junction (at 165.1 68.58) (diameter 0) (color 0 0 0 0)
+  )
+  (junction (at 116.84 53.34) (diameter 0) (color 0 0 0 0)
   )
   (junction (at 170.18 121.92) (diameter 0) (color 0 0 0 0)
@@
   (junction (at 116.84 66.04) (diameter 0) (color 0 0 0 0)
   )
+  (junction (at 139.7 53.34) (diameter 0) (color 0 0 0 0)
+  )
   (junction (at 149.86 100.33) (diameter 0) (color 0 0 0 0)
   )
@@
   (junction (at 170.18 110.49) (diameter 0) (color 0 0 0 0)
   )
-  (junction (at 116.84 49.53) (diameter 0) (color 0 0 0 0)
-  )
-  (junction (at 139.7 49.53) (diameter 0) (color 0 0 0 0)
-  )
   (junction (at 139.7 143.51) (diameter 0) (color 0 0 0 0)
   )
@@
     (stroke (width 0) (type default))
   )
-  (wire (pts (xy 165.1 69.85) (xy 165.1 71.12))
+  (wire (pts (xy 165.1 67.31) (xy 165.1 68.58))
     (stroke (width 0) (type default))
   )
@@
     (stroke (width 0) (type default))
   )
-  (wire (pts (xy 116.84 55.88) (xy 116.84 49.53))
+  (wire (pts (xy 116.84 55.88) (xy 116.84 53.34))
     (stroke (width 0) (type default))
   )
@@
     (stroke (width 0) (type default))
   )
-  (wire (pts (xy 139.7 48.26) (xy 139.7 49.53))
-    (stroke (width 0) (type default))
-  )
   (wire (pts (xy 139.7 133.35) (xy 154.94 133.35))
     (stroke (width 0) (type default))
@@
     (stroke (width 0) (type default))
   )
-  (wire (pts (xy 165.1 58.42) (xy 165.1 62.23))
-    (stroke (width 0) (type default))
-  )
-  (wire (pts (xy 165.1 58.42) (xy 139.7 58.42))
+  (wire (pts (xy 165.1 53.34) (xy 165.1 59.69))
+    (stroke (width 0) (type default))
+  )
+  (wire (pts (xy 165.1 53.34) (xy 139.7 53.34))
     (stroke (width 0) (type default))
   )
@@
     (stroke (width 0) (type default))
   )
-  (wire (pts (xy 165.1 71.12) (xy 168.91 71.12))
+  (wire (pts (xy 165.1 68.58) (xy 168.91 68.58))
     (stroke (width 0) (type default))
   )
@@
     (stroke (width 0) (type default))
   )
-  (wire (pts (xy 116.84 49.53) (xy 139.7 49.53))
-    (stroke (width 0) (type default))
-  )
   (wire (pts (xy 95.25 81.28) (xy 101.6 81.28))
     (stroke (width 0) (type default))
   )
-  (wire (pts (xy 107.95 49.53) (xy 107.95 54.61))
+  (wire (pts (xy 107.95 53.34) (xy 107.95 54.61))
     (stroke (width 0) (type default))
   )
@@
     (stroke (width 0) (type default))
   )
-  (wire (pts (xy 139.7 58.42) (xy 139.7 60.96))
+  (wire (pts (xy 139.7 53.34) (xy 139.7 60.96))
     (stroke (width 0) (type default))
   )
@@
     (stroke (width 0) (type default))
   )
+  (wire (pts (xy 139.7 53.34) (xy 116.84 53.34))
+    (stroke (width 0) (type default))
+  )
   (wire (pts (xy 179.07 100.33) (xy 179.07 121.92))
     (stroke (width 0) (type default))
@@
     (stroke (width 0) (type default))
   )
-  (wire (pts (xy 165.1 80.01) (xy 165.1 83.82))
+  (wire (pts (xy 165.1 77.47) (xy 165.1 83.82))
     (stroke (width 0) (type default))
   )
@@
     (stroke (width 0) (type default))
   )
-  (wire (pts (xy 168.91 49.53) (xy 168.91 71.12))
+  (wire (pts (xy 168.91 46.99) (xy 168.91 68.58))
     (stroke (width 0) (type default))
   )
@@
     (stroke (width 0) (type default))
   )
-  (wire (pts (xy 165.1 71.12) (xy 165.1 72.39))
+  (wire (pts (xy 165.1 68.58) (xy 165.1 69.85))
     (stroke (width 0) (type default))
   )
@@
     (stroke (width 0) (type default))
   )
-  (wire (pts (xy 139.7 49.53) (xy 168.91 49.53))
-    (stroke (width 0) (type default))
-  )
   (wire (pts (xy 90.17 81.28) (xy 95.25 81.28))
     (stroke (width 0) (type default))
@@
     (stroke (width 0) (type default))
   )
-  (wire (pts (xy 116.84 49.53) (xy 107.95 49.53))
+  (wire (pts (xy 116.84 53.34) (xy 107.95 53.34))
     (stroke (width 0) (type default))
   )
@@
     (effects (font (size 2.5 2.5)) (justify left bottom))
   )
-  (text "BYPASS\nFUSE" (at 154.94 78.74 0)
+  (text "BYPASS\nFUSE" (at 154.94 76.2 0)
     (effects (font (size 1.27 1.27)) (justify left bottom))
   )
@@
       (effects (font (size 1.27 1.27)))
     )
-    (property "Value" "1k" (at 104.14 77.47 90)
+    (property "Value" "220" (at 104.14 77.47 90)
       (effects (font (size 1.27 1.27)))
     )
@@
     )
   )
-  (symbol (lib_id "gnarboard:ATC Fuse Bypass") (at 165.1 71.12 0) (unit 1)
+  (symbol (lib_id "gnarboard:ATC Fuse Bypass") (at 165.1 68.58 0) (unit 1)
     (in_bom yes) (on_board yes) (dnp no)
-    (property "Reference" "F1" (at 157.48 64.77 0)
-      (effects (font (size 1.27 1.27)) (justify left))
-    )
-    (property "Value" "25A" (at 157.48 67.31 0)
-      (effects (font (size 1.27 1.27)) (justify left))
-    )
-    (property "Footprint" "gnarboard:ATC Bypass Fuse" (at 162.052 67.31 90)
-      (effects (font (size 1.27 1.27)) hide)
-    )
-    (property "Datasheet" "~" (at 163.83 67.31 0)
-      (effects (font (size 1.27 1.27)) hide)
-    )
-    (property "Vendor" "833-GS1G-LTP" (at 165.1 71.12 0)
+    (property "Reference" "F1" (at 157.48 62.23 0)
+      (effects (font (size 1.27 1.27)) (justify left))
+    )
+    (property "Value" "25A" (at 157.48 64.77 0)
+      (effects (font (size 1.27 1.27)) (justify left))
+    )
+    (property "Footprint" "gnarboard:ATC Bypass Fuse" (at 162.052 64.77 90)
+      (effects (font (size 1.27 1.27)) hide)
+    )
+    (property "Datasheet" "~" (at 163.83 64.77 0)
+      (effects (font (size 1.27 1.27)) hide)
+    )
+    (property "Vendor" "833-GS1G-LTP" (at 165.1 68.58 0)
       (effects (font (size 1.27 1.27)) hide)
     )
@@
     )
   )
-  (symbol (lib_id "power:+24V") (at 139.7 48.26 0) (unit 1)
-    (in_bom yes) (on_board yes) (dnp no) (fields_autoplaced)
-    (property "Reference" "#PWR015" (at 139.7 52.07 0)
-      (effects (font (size 1.27 1.27)) hide)
-    )
-    (property "Value" "+24V" (at 139.7 43.18 0)
+  (symbol (lib_id "power:+24V") (at 168.91 46.99 0) (unit 1)
+    (in_bom yes) (on_board yes) (dnp no) (fields_autoplaced)
+    (property "Reference" "#PWR015" (at 168.91 50.8 0)
+      (effects (font (size 1.27 1.27)) hide)
+    )
+    (property "Value" "+24V" (at 168.91 41.91 0)
       (effects (font (size 1.27 1.27)))
     )
-    (property "Footprint" "" (at 139.7 48.26 0)
-      (effects (font (size 1.27 1.27)) hide)
-    )
-    (property "Datasheet" "" (at 139.7 48.26 0)
+    (property "Footprint" "" (at 168.91 46.99 0)
+      (effects (font (size 1.27 1.27)) hide)
+    )
+    (property "Datasheet" "" (at 168.91 46.99 0)
       (effects (font (size 1.27 1.27)) hide)
     )
@@
     )
   )
-  (symbol (lib_id "Transistor_BJT:BC817") (at 114.3 81.28 0) (unit 1)
+  (symbol (lib_id "Transistor_FET:2N7002") (at 114.3 81.28 0) (unit 1)
     (in_bom yes) (on_board yes) (dnp no)
     (property "Reference" "Q2" (at 119.38 80.01 0)
       (effects (font (size 1.27 1.27)) (justify left))
     )
-    (property "Value" "BC817" (at 119.38 82.55 0)
+    (property "Value" "2N7002" (at 119.38 82.55 0)
       (effects (font (size 1.27 1.27)) (justify left))
     )
@@
       (effects (font (size 1.27 1.27) italic) (justify left) hide)
     )
-    (property "Datasheet" "https://www.onsemi.com/pub/Collateral/BC818-D.pdf" (at 114.3 81.28 0)
+    (property "Datasheet" "https://www.onsemi.com/pub/Collateral/NDS7002A-D.PDF" (at 114.3 81.28 0)
       (effects (font (size 1.27 1.27)) (justify left) hide)
     )
