File: boards/8ch-mosfet/mosfet.kicad_sch (KiCad schematic)
At the start: 15 parts, among them J5 Screw_Terminal_01x02, Q1 IRF4905, Q2 2N7002, U5 ACS725xLCTR-20AU

Commit message: updated layout with new fuse.
Parts:
- F1: footprint gnarboard:ATC Bypass Fuse -> yarrboard:ATC Bypass Fuse
- J5: footprint gnarboard:Molex 1x02 .375 -> yarrboard:Molex 1x02 .375
- U5: footprint gnarboard:ACS7XX -> yarrboard:ACS7XX
Changed lines of the file:
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@@
       (effects (font (size 1.27 1.27)) (justify left))
     )
-    (property "Footprint" "gnarboard:ATC Bypass Fuse" (at 162.052 64.77 90)
+    (property "Footprint" "yarrboard:ATC Bypass Fuse" (at 162.052 64.77 90)
       (effects (font (size 1.27 1.27)) hide)
     )
@@
       (effects (font (size 1.27 1.27)) (justify left) hide)
     )
-    (property "Footprint" "gnarboard:Molex 1x02 .375" (at 160.02 137.16 0)
+    (property "Footprint" "yarrboard:Molex 1x02 .375" (at 160.02 137.16 0)
       (effects (font (size 1.27 1.27)) hide)
     )
@@
       (effects (font (size 1.27 1.27)) (justify left) hide)
     )
-    (property "Footprint" "gnarboard:ACS7XX" (at 152.4 119.38 0)
+    (property "Footprint" "yarrboard:ACS7XX" (at 152.4 119.38 0)
       (effects (font (size 1.27 1.27) italic) (justify left) hide)
     )

Commit message: prepared 8ch mosfet for production
Other:
- company: (none) -> https://github.com/hoeken/yarrboard
- title: (none) -> Yarrboard 8ch Mosfet Driver
Changed lines of the file:
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@@
 (kicad_sch (version 20230121) (generator eeschema)
   (paper "A4")
+  (title_block
+    (title "Yarrboard 8ch Mosfet Driver")
+    (company "https://github.com/hoeken/yarrboard")
+  )
   (junction (at 165.1 68.58) (diameter 0) (color 0 0 0 0)
   )

Commit message: updated BOM
Parts:
- C3: Mouser (none) -> C0805C102J1HACTU; Vendor C0805C102J1HACTU -> (none)
- C4: Mouser (none) -> C0805C472K5RAC; Vendor C0805C472K5RAC -> (none)
- C5: Mouser (none) -> 08053C104KAT4A; Vendor 08053C104KAT4A -> (none)
- D10: Mouser (none) -> 625-SS16-E3; Vendor 625-SS16-E3 -> (none)
- D18: Mouser (none) -> 771-BZX384-C15115; Vendor 771-BZX384-C15115 -> (none)
- D2: Mouser (none) -> 150080RS75000; Vendor 150080RS75000 -> (none)
- F1: Mouser (none) -> 534-3522-3; Vendor 833-GS1G-LTP -> (none)
- J5: JCLC (none) -> JL45C-09516B01; Mouser (none) -> 538-38720-7516; Vendor OQ0271500000G, TJ0271500000G -> (none)
- Q1: Mouser (none) -> 942-IRF4905STRLPBF; Vendor 942-IRF4905STRLPBF -> (none)
- Q2: Mouser (none) -> 771-BC817-25-T/R; Vendor 771-BC817-25-T/R -> (none)
- R1: value 220 -> 220R; Vendor 652-CR0805JW-103ELF -> (none)
- R2: Vendor 652-CR0805JW-102ELF -> (none)
- R3: Vendor 652-CR0805JW-472ELF -> (none)
- R4: Vendor 652-CR0805JW-223ELF -> (none)
- U5: Mouser (none) -> 250-725LLCTR20AUT; Vendor 250-725LLCTR20AUT -> (none)
Other:
- moved on the sheet: C4
Changed lines of the file:
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@@
     (stroke (width 0) (type default))
   )
-  (wire (pts (xy 170.18 110.49) (xy 170.18 113.03))
+  (wire (pts (xy 170.18 110.49) (xy 170.18 114.3))
     (stroke (width 0) (type default))
   )
@@
     (stroke (width 0) (type default))
   )
-  (wire (pts (xy 170.18 118.11) (xy 170.18 121.92))
+  (wire (pts (xy 170.18 119.38) (xy 170.18 121.92))
     (stroke (width 0) (type default))
   )
@@
       (effects (font (size 1.27 1.27)))
     )
-    (property "Value" "220" (at 104.14 77.47 90)
+    (property "Value" "220R" (at 104.14 77.47 90)
       (effects (font (size 1.27 1.27)))
     )
@@
       (effects (font (size 1.27 1.27)) hide)
     )
-    (property "Vendor" " 652-CR0805JW-103ELF " (at 104.14 81.28 0)
-      (effects (font (size 1.27 1.27)) hide)
-    )
     (pin "1")
     (pin "2")
@@
       (effects (font (size 1.27 1.27)) hide)
     )
-    (property "Vendor" "625-SS16-E3 " (at 139.7 138.43 0)
+    (property "Mouser" "625-SS16-E3 " (at 139.7 138.43 0)
       (effects (font (size 1.27 1.27)) hide)
     )
@@
       (effects (font (size 1.27 1.27)) hide)
     )
-    (property "Vendor" " 652-CR0805JW-102ELF " (at 95.25 85.09 0)
-      (effects (font (size 1.27 1.27)) hide)
-    )
     (pin "1")
     (pin "2")
@@
     )
     (property "Datasheet" "~" (at 116.84 58.42 0)
-      (effects (font (size 1.27 1.27)) hide)
-    )
-    (property "Vendor" " 652-CR0805JW-223ELF " (at 116.84 58.42 0)
       (effects (font (size 1.27 1.27)) hide)
     )
@@
       (effects (font (size 1.27 1.27)) hide)
     )
-    (property "Vendor" "833-GS1G-LTP" (at 165.1 68.58 0)
+    (property "Mouser" "534-3522-3 " (at 165.1 68.58 0)
       (effects (font (size 1.27 1.27)) hide)
     )
@@
       (effects (font (size 1.27 1.27)) hide)
     )
-    (property "Vendor" "150080RS75000" (at 95.25 91.44 0)
+    (property "Mouser" "150080RS75000" (at 95.25 91.44 0)
       (effects (font (size 1.27 1.27)) hide)
     )
@@
       (effects (font (size 1.27 1.27)) hide)
     )
-    (property "Vendor" "08053C104KAT4A" (at 166.37 100.33 0)
+    (property "Mouser" "08053C104KAT4A" (at 166.37 100.33 0)
       (effects (font (size 1.27 1.27)) hide)
     )
@@
     )
   )
-  (symbol (lib_id "Device:C_Small") (at 170.18 115.57 0) (unit 1)
-    (in_bom yes) (on_board yes) (dnp no) (fields_autoplaced)
-    (property "Reference" "C4" (at 172.72 114.3063 0)
-      (effects (font (size 1.27 1.27)) (justify left))
-    )
-    (property "Value" "4.7nF" (at 172.72 116.8463 0)
-      (effects (font (size 1.27 1.27)) (justify left))
-    )
-    (property "Footprint" "Capacitor_SMD:C_0805_2012Metric_Pad1.18x1.45mm_HandSolder" (at 170.18 115.57 0)
-      (effects (font (size 1.27 1.27)) hide)
-    )
-    (property "Datasheet" "~" (at 170.18 115.57 0)
-      (effects (font (size 1.27 1.27)) hide)
-    )
-    (property "Vendor" "C0805C472K5RAC" (at 170.18 115.57 0)
+  (symbol (lib_id "Device:C_Small") (at 170.18 116.84 0) (unit 1)
+    (in_bom yes) (on_board yes) (dnp no) (fields_autoplaced)
+    (property "Reference" "C4" (at 172.72 115.5763 0)
+      (effects (font (size 1.27 1.27)) (justify left))
+    )
+    (property "Value" "4.7nF" (at 172.72 118.1163 0)
+      (effects (font (size 1.27 1.27)) (justify left))
+    )
+    (property "Footprint" "Capacitor_SMD:C_0805_2012Metric_Pad1.18x1.45mm_HandSolder" (at 170.18 116.84 0)
+      (effects (font (size 1.27 1.27)) hide)
+    )
+    (property "Datasheet" "~" (at 170.18 116.84 0)
+      (effects (font (size 1.27 1.27)) hide)
+    )
+    (property "Mouser" "C0805C472K5RAC" (at 170.18 116.84 0)
       (effects (font (size 1.27 1.27)) hide)
     )
@@
       (effects (font (size 1.27 1.27)) hide)
     )
-    (property "Vendor" "OQ0271500000G, TJ0271500000G" (at 160.02 137.16 0)
+    (property "Mouser" " 538-38720-7516" (at 160.02 137.16 0)
+      (effects (font (size 1.27 1.27)) hide)
+    )
+    (property "JCLC" "JL45C-09516B01" (at 160.02 137.16 0)
       (effects (font (size 1.27 1.27)) hide)
     )
@@
       (effects (font (size 1.27 1.27)) hide)
     )
-    (property "Vendor" "250-725LLCTR20AUT" (at 149.86 110.49 0)
+    (property "Mouser" "250-725LLCTR20AUT" (at 149.86 110.49 0)
       (effects (font (size 1.27 1.27)) hide)
     )
@@
       (effects (font (size 1.27 1.27)) hide)
     )
-    (property "Vendor" "652-CR0805JW-472ELF" (at 116.84 71.12 0)
-      (effects (font (size 1.27 1.27)) hide)
-    )
     (pin "1")
     (pin "2")
@@
       (effects (font (size 1.27 1.27)) hide)
     )
-    (property "Vendor" "C0805C102J1HACTU" (at 161.29 116.84 0)
+    (property "Mouser" "C0805C102J1HACTU" (at 161.29 116.84 0)
       (effects (font (size 1.27 1.27)) hide)
     )
@@
       (effects (font (size 1.27 1.27)) hide)
     )
-    (property "Vendor" "771-BZX384-C15115" (at 107.95 58.42 90)
+    (property "Mouser" "771-BZX384-C15115" (at 107.95 58.42 90)
       (effects (font (size 1.27 1.27)) hide)
     )
@@
       (effects (font (size 1.27 1.27)) (justify left) hide)
     )
-    (property "Vendor" " 942-IRF4905STRLPBF " (at 137.16 66.04 0)
+    (property "Mouser" " 942-IRF4905STRLPBF " (at 137.16 66.04 0)
       (effects (font (size 1.27 1.27)) hide)
     )
@@
       (effects (font (size 1.27 1.27)) (justify left) hide)
     )
-    (property "Vendor" "771-BC817-25-T/R" (at 114.3 81.28 0)
-      (effects (font (size 1.27 1.27)) hide)
-    )
+    (property "Mouser" "771-BC817-25-T/R" (at 114.3 81.28 0)
+      (effects (font (size 1.27 1.27)) hide)
+    )

Commit message: more BOM updates.
Parts:
- C3: LCSC (none) -> C94121
- C4: LCSC (none) -> C107153
- C5: LCSC (none) -> C49678
- R1: LCSC (none) -> C114519
- R2: LCSC (none) -> C95781
- R3: LCSC (none) -> C114565
- R4: LCSC (none) -> C96346
Changed lines of the file:
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@@
+      (effects (font (size 1.27 1.27)) hide)
+    )
+    (property "LCSC" "C114519" (at 104.14 81.28 90)
       (effects (font (size 1.27 1.27)) hide)
     )
@@
       (effects (font (size 1.27 1.27)) hide)
     )
+    (property "LCSC" "C95781" (at 95.25 85.09 0)
+      (effects (font (size 1.27 1.27)) hide)
+    )
     (pin "1")
     (pin "2")
@@
     )
     (property "Datasheet" "~" (at 116.84 58.42 0)
+      (effects (font (size 1.27 1.27)) hide)
+    )
+    (property "LCSC" "C96346" (at 116.84 58.42 0)
       (effects (font (size 1.27 1.27)) hide)
     )
@@
       (effects (font (size 1.27 1.27)) hide)
     )
+    (property "LCSC" "C49678" (at 166.37 100.33 90)
+      (effects (font (size 1.27 1.27)) hide)
+    )
     (pin "1")
     (pin "2")
@@
     )
     (property "Mouser" "C0805C472K5RAC" (at 170.18 116.84 0)
+      (effects (font (size 1.27 1.27)) hide)
+    )
+    (property "LCSC" "C107153" (at 170.18 116.84 0)
       (effects (font (size 1.27 1.27)) hide)
     )
@@
       (effects (font (size 1.27 1.27)) hide)
     )
+    (property "LCSC" "C114565" (at 116.84 71.12 0)
+      (effects (font (size 1.27 1.27)) hide)
+    )
     (pin "1")
     (pin "2")
@@
       (effects (font (size 1.27 1.27)) hide)
     )
+    (property "LCSC" "C94121" (at 161.29 116.84 0)
+      (effects (font (size 1.27 1.27)) hide)
+    )

Commit message: removed mouser p/n
Parts:
- Q2: Mouser 771-BC817-25-T/R -> ?????
Changed lines of the file:
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@@
       (effects (font (size 1.27 1.27)) (justify left) hide)
     )
-    (property "Mouser" "771-BC817-25-T/R" (at 114.3 81.28 0)
+    (property "Mouser" "?????" (at 114.3 81.28 0)
       (effects (font (size 1.27 1.27)) hide)
     )
