File: boards/8ch-mosfet/pwm fan.kicad_sch (KiCad schematic)
At the start: 4 parts, among them M1 Fan_4pin

Commit message: updated layout with new fuse.
Parts:
- M1: footprint gnarboard:Molex 0470531000 -> yarrboard:Molex 0470531000
Changed lines of the file:
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@@
       (effects (font (size 1.27 1.27)) (justify left))
     )
-    (property "Footprint" "gnarboard:Molex 0470531000" (at 133.35 87.376 0)
+    (property "Footprint" "yarrboard:Molex 0470531000" (at 133.35 87.376 0)
       (effects (font (size 1.27 1.27)) hide)
     )

Commit message: prepared 8ch mosfet for production
Other:
- company: (none) -> https://github.com/hoeken/yarrboard
- title: (none) -> Yarrboard 8ch Mosfet Driver
Changed lines of the file:
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@@
 (kicad_sch (version 20230121) (generator eeschema)
   (paper "A4")
+  (title_block
+    (title "Yarrboard 8ch Mosfet Driver")
+    (company "https://github.com/hoeken/yarrboard")
+  )
   (junction (at 144.78 90.17) (diameter 0) (color 0 0 0 0)
   )

Commit message: updated BOM
Parts:
- D31: LCSC (none) -> C316020
- M1: LCSC (none) -> C3025061; Mouser (none) -> 538-47053-1000; Vendor 538-47053-1000 -> (none)
- R35: Vendor 652-CR0805JW-103ELF -> (none)
Changed lines of the file:
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@@
-      (effects (font (size 1.27 1.27)) hide)
-    )
-    (property "Vendor" "652-CR0805JW-103ELF" (at 156.21 78.74 0)
       (effects (font (size 1.27 1.27)) hide)
     )
@@
       (effects (font (size 1.27 1.27)) hide)
     )
+    (property "LCSC" "C316020" (at 144.78 96.52 90)
+      (effects (font (size 1.27 1.27)) hide)
+    )
     (pin "1")
     (pin "2")
@@
       (effects (font (size 1.27 1.27)) hide)
     )
-    (property "Vendor" "538-47053-1000 " (at 133.35 87.63 0)
+    (property "Mouser" "538-47053-1000 " (at 133.35 87.63 0)
+      (effects (font (size 1.27 1.27)) hide)
+    )
+    (property "LCSC" "C3025061" (at 133.35 87.63 0)
       (effects (font (size 1.27 1.27)) hide)
     )
@@
       (effects (font (size 1.27 1.27)) hide)
     )
+    (property "LCSC" "C316020" (at 152.4 96.52 90)
+      (effects (font (size 1.27 1.27)) hide)
+    )

Commit message: more BOM updates.
Parts:
- R35: LCSC (none) -> C95781
Changed lines of the file:
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@@
+      (effects (font (size 1.27 1.27)) hide)
+    )
+    (property "LCSC" "C95781" (at 156.21 78.74 0)
       (effects (font (size 1.27 1.27)) hide)
     )
