File: boards/8ch-mosfet/untitled2.kicad_sch (KiCad schematic)
At the start: 15 parts, among them J5 Screw_Terminal_01x02, Q1 IRF4905, Q2 2N7002, U5 ACS725xLCTR-20AU

Commit message: worked on the pwm issues
Parts:
- removed C3: 1nF, Capacitor_SMD:C_0805_2012Metric_Pad1.18x1.45mm_HandSolder, symbol Device:C_Small
- removed D18: 15V, Diode_SMD:D_SOD-323_HandSoldering, symbol Device:D_Zener
- removed Q1: IRF4905, Package_TO_SOT_SMD:TO-263-2, symbol Transistor_FET:IRF4905
- removed Q2: 2N7002, Package_TO_SOT_SMD:SOT-23, symbol Transistor_FET:2N7002
- removed R1: 220R, Resistor_SMD:R_0805_2012Metric_Pad1.20x1.40mm_HandSolder, symbol Device:R_Small_US
- removed R2: 1k, Resistor_SMD:R_0805_2012Metric_Pad1.20x1.40mm_HandSolder, symbol Device:R_Small_US
- removed R3: 22K, Resistor_SMD:R_0805_2012Metric_Pad1.20x1.40mm_HandSolder, symbol Device:R_Small_US
- removed R4: 100K, Resistor_SMD:R_0805_2012Metric_Pad1.20x1.40mm_HandSolder, symbol Device:R_Small_US
- added C3: 1uF, Capacitor_SMD:C_0805_2012Metric_Pad1.18x1.45mm_HandSolder, symbol Device:C_Small
- added C3: 1nF, Capacitor_SMD:C_0805_2012Metric_Pad1.18x1.45mm_HandSolder, symbol Device:C_Small
- added Q1: IRFZ44, Package_TO_SOT_SMD:TO-252-2, symbol Transistor_FET:IRLZ44N
- added R2 (x2): 0, Resistor_SMD:R_0805_2012Metric_Pad1.20x1.40mm_HandSolder, symbol Device:R_Small_US
- added R2: 1k, Resistor_SMD:R_0805_2012Metric_Pad1.20x1.40mm_HandSolder, symbol Device:R_Small_US
- added U16: ~, Package_SO:SOIC-8_3.9x4.9mm_P1.27mm, symbol yarrboard:TC4432
Connections:
- net GNDA: now also C3.2
- net GNDPWR: now also C3.2, U16.4 (GND), U16.5 (GND)
- net PWM: now also R2.2, U16.2 (IN)
- net at D2.2 (A): now also R2.1
- net at F1.1: now also C3.1, Q1.2 (D), U16.1 (VDD)
- net at F1.3, U5.1 (IP+), U5.2 (IP+): now also Q1.3 (S)
- net at U5.6 (FILTER): now also C3.1
- new net: R2.2, U16.6 (OUT)
- new net: R2.2, U16.7 (OUT)
- new net: Q1.1 (G), R2.1, R2.1
- no-connect marks 0 -> 1
Other:
- note added: "Gate Driver"
- note added: "Output Connector"
- note removed: "MOSFET Driver"
- company: https://github.com/hoeken/yarrboard -> (none)
- title: Yarrboard 8ch Mosfet Driver -> (none)

Commit message: starting a redesign ahead of having parts to test. wish me luck
Connections:
- net at C3.1, F1.1, Q1.2 (D)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: now also U16.8 (VDD)
Changed lines of the file:
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@@
   (junction (at 143.51 130.81) (diameter 0) (color 0 0 0 0)
+  )
+  (junction (at 128.27 50.8) (diameter 0) (color 0 0 0 0)
   )
   (junction (at 143.51 140.97) (diameter 0) (color 0 0 0 0)
@@
   )
   (wire (pts (xy 102.87 90.17) (xy 102.87 140.97))
+    (stroke (width 0) (type default))
+  )
+  (wire (pts (xy 128.27 59.69) (xy 128.27 50.8))
     (stroke (width 0) (type default))
   )
@@
     (stroke (width 0) (type default))
   )
+  (wire (pts (xy 125.73 59.69) (xy 128.27 59.69))
+    (stroke (width 0) (type default))
+  )
   (wire (pts (xy 163.83 105.41) (xy 173.99 105.41))
     (stroke (width 0) (type default))
   )
-  (wire (pts (xy 143.51 50.8) (xy 102.87 50.8))
+  (wire (pts (xy 143.51 50.8) (xy 128.27 50.8))
     (stroke (width 0) (type default))
   )
@@
     (stroke (width 0) (type default))
   )
+  (wire (pts (xy 128.27 50.8) (xy 102.87 50.8))
+    (stroke (width 0) (type default))
+  )
