File: boards/8ch-mosfet/connectors.kicad_sch (KiCad schematic)
At the start: 10 parts, among them J1 N2K, J2 I2C

Commit message: more BOM updates.
Parts:
- J1: now not fitted; now left out of the parts list
Changed lines of the file:
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@@
   )
   (symbol (lib_id "Connector_Generic:Conn_01x04") (at 35.56 81.28 0) (mirror y) (unit 1)
-    (in_bom yes) (on_board yes) (dnp no) (fields_autoplaced)
+    (in_bom no) (on_board yes) (dnp yes) (fields_autoplaced)
     (property "Reference" "J1" (at 33.02 81.28 0)
       (effects (font (size 1.27 1.27)) (justify left))
