File: boards/button pad board/button pad board.kicad_sch (KiCad schematic)
At the start: 1 part, among them SW1 SW_Push

Commit message: oh yeah, looking good.
Parts:
- removed SW1: SW_Push, symbol Switch:SW_Push
- added U1, U2, U3, U4: ~, yarrboard:BUTTONPAD-2X2, symbol yarrboard:2x2_RGB_Button
Connections:
- new net +5V: U1.VCC, U1.VCC, U2.VCC, U2.VCC, U3.VCC, U3.VCC, U4.VCC, U4.VCC
- new net B0: U1.B1, U2.B1, U3.B1, U4.B1
- new net B1: U1.B2, U2.B2, U3.B2, U4.B2
- new net B2: U1.B3, U2.B3, U3.B3, U4.B3
- new net B3: U1.B4, U2.B4, U3.B4, U4.B4
- new net G0: U1.G1, U2.G1, U3.G1, U4.G1
- new net G1: U1.G2, U2.G2, U3.G2, U4.G2
- new net G2: U1.G3, U2.G3, U3.G3, U4.G3
- new net G3: U1.G4, U2.G4, U3.G4, U4.G4
- new net GND: U1.SWB1, U1.SWB1, U1.SWB2, U1.SWB3, U1.SWB4, U2.SWB1, U2.SWB1, U2.SWB2, U2.SWB3, U2.SWB4, U3.SWB1, U3.SWB1, U3.SWB2, U3.SWB3, U3.SWB4, U4.SWB1, U4.SWB1, U4.SWB2, U4.SWB3, U4.SWB4
- new net IN0: U1.SWA1, U2.SWA1, U3.SWA1, U4.SWA1
- new net IN1: U1.SWA2, U2.SWA2, U3.SWA2, U4.SWA2
- new net IN2: U1.SWA3, U2.SWA3, U3.SWA3, U4.SWA3
- new net IN3: U1.SWA4, U2.SWA4, U3.SWA4, U4.SWA4
- new net R0: U1.R1, U2.R1, U3.R1, U4.R1
- new net R1: U1.R2, U2.R2, U3.R2, U4.R2
- new net R2: U1.R3, U2.R3, U3.R3, U4.R3
- new net R3: U1.R4, U2.R4, U3.R4, U4.R4
- new net VCC: U1.VCC, U1.VCC, U2.VCC, U2.VCC, U3.VCC, U3.VCC, U4.VCC, U4.VCC
