File: boards/button pad board/4x4.kicad_sch (KiCad schematic)
At the start: 5 parts

Commit message: good progress on teh button board
Connections:
- net VCC renamed +5V
Changed lines of the file:
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@@
+    )
+  )
+  (symbol (lib_id "power:+5V") (at 139.7 59.69 0) (unit 1)
+    (in_bom yes) (on_board yes) (dnp no) (fields_autoplaced)
+    (property "Reference" "#PWR01" (at 139.7 63.5 0)
+      (effects (font (size 1.27 1.27)) hide)
+    )
+    (property "Value" "+5V" (at 139.7 54.61 0)
+      (effects (font (size 1.27 1.27)))
+    )
+    (property "Footprint" "" (at 139.7 59.69 0)
+      (effects (font (size 1.27 1.27)) hide)
+    )
+    (property "Datasheet" "" (at 139.7 59.69 0)
+      (effects (font (size 1.27 1.27)) hide)
+    )
+    (pin "1")
+    (instances
+      (project "button pad board"
+        (path "/66d98af2-097e-4f68-99f2-351c9b9568f9/544cec96-03d5-4637-ae41-3c1a8e8dda15"
+          (reference "#PWR01") (unit 1)
+        )
+        (path "/66d98af2-097e-4f68-99f2-351c9b9568f9/edbb582d-fe2b-48b6-8d6d-cfd6eb008018"
+          (reference "#PWR02") (unit 1)
+        )
+        (path "/66d98af2-097e-4f68-99f2-351c9b9568f9/d32bb895-5dd5-4c02-b031-f9ed3ff2fbb5"
+          (reference "#PWR05") (unit 1)
+        )
+        (path "/66d98af2-097e-4f68-99f2-351c9b9568f9/214ea90b-349a-415c-a8ca-f88377356f85"
+          (reference "#PWR06") (unit 1)
+        )
+      )
     )
   )
@@
     )
   )
-  (symbol (lib_id "power:VCC") (at 166.37 97.79 0) (unit 1)
-    (in_bom yes) (on_board yes) (dnp no) (fields_autoplaced)
-    (property "Reference" "#PWR03" (at 166.37 101.6 0)
-      (effects (font (size 1.27 1.27)) hide)
-    )
-    (property "Value" "VCC" (at 166.37 92.71 0)
-      (effects (font (size 1.27 1.27)))
-    )
-    (property "Footprint" "" (at 166.37 97.79 0)
-      (effects (font (size 1.27 1.27)) hide)
-    )
-    (property "Datasheet" "" (at 166.37 97.79 0)
-      (effects (font (size 1.27 1.27)) hide)
-    )
-    (pin "1")
-    (instances
-      (project "button pad board"
-        (path "/66d98af2-097e-4f68-99f2-351c9b9568f9"
-          (reference "#PWR03") (unit 1)
-        )
-        (path "/66d98af2-097e-4f68-99f2-351c9b9568f9/544cec96-03d5-4637-ae41-3c1a8e8dda15"
-          (reference "#PWR06") (unit 1)
-        )
-        (path "/66d98af2-097e-4f68-99f2-351c9b9568f9/edbb582d-fe2b-48b6-8d6d-cfd6eb008018"
-          (reference "#PWR014") (unit 1)
-        )
-        (path "/66d98af2-097e-4f68-99f2-351c9b9568f9/d32bb895-5dd5-4c02-b031-f9ed3ff2fbb5"
-          (reference "#PWR022") (unit 1)
-        )
-        (path "/66d98af2-097e-4f68-99f2-351c9b9568f9/214ea90b-349a-415c-a8ca-f88377356f85"
-          (reference "#PWR030") (unit 1)
-        )
-      )
-    )
-  )
   (symbol (lib_id "power:GND") (at 166.37 118.11 0) (unit 1)
     (in_bom yes) (on_board yes) (dnp no) (fields_autoplaced)
@@
     )
   )
-  (symbol (lib_id "power:VCC") (at 139.7 97.79 0) (unit 1)
-    (in_bom yes) (on_board yes) (dnp no) (fields_autoplaced)
-    (property "Reference" "#PWR04" (at 139.7 101.6 0)
-      (effects (font (size 1.27 1.27)) hide)
-    )
-    (property "Value" "VCC" (at 139.7 92.71 0)
-      (effects (font (size 1.27 1.27)))
-    )
-    (property "Footprint" "" (at 139.7 97.79 0)
-      (effects (font (size 1.27 1.27)) hide)
-    )
-    (property "Datasheet" "" (at 139.7 97.79 0)
-      (effects (font (size 1.27 1.27)) hide)
-    )
-    (pin "1")
-    (instances
-      (project "button pad board"
-        (path "/66d98af2-097e-4f68-99f2-351c9b9568f9"
-          (reference "#PWR04") (unit 1)
-        )
-        (path "/66d98af2-097e-4f68-99f2-351c9b9568f9/544cec96-03d5-4637-ae41-3c1a8e8dda15"
-          (reference "#PWR05") (unit 1)
-        )
-        (path "/66d98af2-097e-4f68-99f2-351c9b9568f9/edbb582d-fe2b-48b6-8d6d-cfd6eb008018"
-          (reference "#PWR013") (unit 1)
+  (symbol (lib_id "power:+5V") (at 166.37 97.79 0) (unit 1)
+    (in_bom yes) (on_board yes) (dnp no) (fields_autoplaced)
+    (property "Reference" "#PWR017" (at 166.37 101.6 0)
+      (effects (font (size 1.27 1.27)) hide)
+    )
+    (property "Value" "+5V" (at 166.37 92.71 0)
+      (effects (font (size 1.27 1.27)))
+    )
+    (property "Footprint" "" (at 166.37 97.79 0)
+      (effects (font (size 1.27 1.27)) hide)
+    )
+    (property "Datasheet" "" (at 166.37 97.79 0)
+      (effects (font (size 1.27 1.27)) hide)
+    )
+    (pin "1")
+    (instances
+      (project "button pad board"
+        (path "/66d98af2-097e-4f68-99f2-351c9b9568f9/544cec96-03d5-4637-ae41-3c1a8e8dda15"
+          (reference "#PWR017") (unit 1)
+        )
+        (path "/66d98af2-097e-4f68-99f2-351c9b9568f9/edbb582d-fe2b-48b6-8d6d-cfd6eb008018"
+          (reference "#PWR018") (unit 1)
         )
         (path "/66d98af2-097e-4f68-99f2-351c9b9568f9/d32bb895-5dd5-4c02-b031-f9ed3ff2fbb5"
@@
         )
         (path "/66d98af2-097e-4f68-99f2-351c9b9568f9/214ea90b-349a-415c-a8ca-f88377356f85"
-          (reference "#PWR029") (unit 1)
-        )
-      )
-    )
-  )
-  (symbol (lib_id "power:VCC") (at 166.37 59.69 0) (unit 1)
-    (in_bom yes) (on_board yes) (dnp no) (fields_autoplaced)
-    (property "Reference" "#PWR02" (at 166.37 63.5 0)
-      (effects (font (size 1.27 1.27)) hide)
-    )
-    (property "Value" "VCC" (at 166.37 54.61 0)
-      (effects (font (size 1.27 1.27)))
-    )
-    (property "Footprint" "" (at 166.37 59.69 0)
-      (effects (font (size 1.27 1.27)) hide)
-    )
-    (property "Datasheet" "" (at 166.37 59.69 0)
-      (effects (font (size 1.27 1.27)) hide)
-    )
-    (pin "1")
-    (instances
-      (project "button pad board"
-        (path "/66d98af2-097e-4f68-99f2-351c9b9568f9"
-          (reference "#PWR02") (unit 1)
-        )
-        (path "/66d98af2-097e-4f68-99f2-351c9b9568f9/544cec96-03d5-4637-ae41-3c1a8e8dda15"
-          (reference "#PWR02") (unit 1)
-        )
-        (path "/66d98af2-097e-4f68-99f2-351c9b9568f9/edbb582d-fe2b-48b6-8d6d-cfd6eb008018"
-          (reference "#PWR010") (unit 1)
-        )
-        (path "/66d98af2-097e-4f68-99f2-351c9b9568f9/d32bb895-5dd5-4c02-b031-f9ed3ff2fbb5"
-          (reference "#PWR018") (unit 1)
-        )
-        (path "/66d98af2-097e-4f68-99f2-351c9b9568f9/214ea90b-349a-415c-a8ca-f88377356f85"
-          (reference "#PWR026") (unit 1)
+          (reference "#PWR022") (unit 1)
         )
       )
@@
     )
   )
-  (symbol (lib_id "power:VCC") (at 139.7 59.69 0) (unit 1)
-    (in_bom yes) (on_board yes) (dnp no) (fields_autoplaced)
-    (property "Reference" "#PWR01" (at 139.7 63.5 0)
-      (effects (font (size 1.27 1.27)) hide)
-    )
-    (property "Value" "VCC" (at 139.7 54.61 0)
-      (effects (font (size 1.27 1.27)))
-    )
-    (property "Footprint" "" (at 139.7 59.69 0)
-      (effects (font (size 1.27 1.27)) hide)
-    )
-    (property "Datasheet" "" (at 139.7 59.69 0)
-      (effects (font (size 1.27 1.27)) hide)
-    )
-    (pin "1")
-    (instances
-      (project "button pad board"
-        (path "/66d98af2-097e-4f68-99f2-351c9b9568f9"
-          (reference "#PWR01") (unit 1)
-        )
-        (path "/66d98af2-097e-4f68-99f2-351c9b9568f9/544cec96-03d5-4637-ae41-3c1a8e8dda15"
-          (reference "#PWR01") (unit 1)
-        )
-        (path "/66d98af2-097e-4f68-99f2-351c9b9568f9/edbb582d-fe2b-48b6-8d6d-cfd6eb008018"
+  (symbol (lib_id "power:+5V") (at 139.7 97.79 0) (unit 1)
+    (in_bom yes) (on_board yes) (dnp no) (fields_autoplaced)
+    (property "Reference" "#PWR025" (at 139.7 101.6 0)
+      (effects (font (size 1.27 1.27)) hide)
+    )
+    (property "Value" "+5V" (at 139.7 92.71 0)
+      (effects (font (size 1.27 1.27)))
+    )
+    (property "Footprint" "" (at 139.7 97.79 0)
+      (effects (font (size 1.27 1.27)) hide)
+    )
+    (property "Datasheet" "" (at 139.7 97.79 0)
+      (effects (font (size 1.27 1.27)) hide)
+    )
+    (pin "1")
+    (instances
+      (project "button pad board"
+        (path "/66d98af2-097e-4f68-99f2-351c9b9568f9/544cec96-03d5-4637-ae41-3c1a8e8dda15"
+          (reference "#PWR025") (unit 1)
+        )
+        (path "/66d98af2-097e-4f68-99f2-351c9b9568f9/edbb582d-fe2b-48b6-8d6d-cfd6eb008018"
+          (reference "#PWR026") (unit 1)
+        )
+        (path "/66d98af2-097e-4f68-99f2-351c9b9568f9/d32bb895-5dd5-4c02-b031-f9ed3ff2fbb5"
+          (reference "#PWR029") (unit 1)
+        )
+        (path "/66d98af2-097e-4f68-99f2-351c9b9568f9/214ea90b-349a-415c-a8ca-f88377356f85"
+          (reference "#PWR030") (unit 1)
+        )
+      )
+    )
+  )
+  (symbol (lib_id "power:+5V") (at 166.37 59.69 0) (unit 1)
+    (in_bom yes) (on_board yes) (dnp no) (fields_autoplaced)
+    (property "Reference" "#PWR09" (at 166.37 63.5 0)
+      (effects (font (size 1.27 1.27)) hide)
+    )
+    (property "Value" "+5V" (at 166.37 54.61 0)
+      (effects (font (size 1.27 1.27)))
+    )
+    (property "Footprint" "" (at 166.37 59.69 0)
+      (effects (font (size 1.27 1.27)) hide)
+    )
+    (property "Datasheet" "" (at 166.37 59.69 0)
+      (effects (font (size 1.27 1.27)) hide)
+    )
+    (pin "1")
+    (instances
+      (project "button pad board"
+        (path "/66d98af2-097e-4f68-99f2-351c9b9568f9/544cec96-03d5-4637-ae41-3c1a8e8dda15"
           (reference "#PWR09") (unit 1)
         )
-        (path "/66d98af2-097e-4f68-99f2-351c9b9568f9/d32bb895-5dd5-4c02-b031-f9ed3ff2fbb5"
-          (reference "#PWR017") (unit 1)
-        )
-        (path "/66d98af2-097e-4f68-99f2-351c9b9568f9/214ea90b-349a-415c-a8ca-f88377356f85"
-          (reference "#PWR025") (unit 1)
-        )
-      )
+        (path "/66d98af2-097e-4f68-99f2-351c9b9568f9/edbb582d-fe2b-48b6-8d6d-cfd6eb008018"
+          (reference "#PWR010") (unit 1)
+        )
+        (path "/66d98af2-097e-4f68-99f2-351c9b9568f9/d32bb895-5dd5-4c02-b031-f9ed3ff2fbb5"
+          (reference "#PWR013") (unit 1)
+        )
+        (path "/66d98af2-097e-4f68-99f2-351c9b9568f9/214ea90b-349a-415c-a8ca-f88377356f85"
+          (reference "#PWR014") (unit 1)
+        )
+      )

Commit message: button board updated, routed, and ready to rock.
Other:
- company: (none) -> github.com/hoeken/yarrboard
- title: (none) -> RGB Button Pad Board
Changed lines of the file:
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@@
 (kicad_sch (version 20230121) (generator eeschema)
   (paper "A4")
+  (title_block
+    (title "RGB Button Pad Board")
+    (rev "Rev A")
+    (company "github.com/hoeken/yarrboard")
+    (comment 1 "Open Source Hardware")
+  )
   (junction (at 162.56 63.5) (diameter 0) (color 0 0 0 0)
   )
@@
         (path "/66d98af2-097e-4f68-99f2-351c9b9568f9/edbb582d-fe2b-48b6-8d6d-cfd6eb008018"
           (reference "#PWR011") (unit 1)
-        )
-        (path "/66d98af2-097e-4f68-99f2-351c9b9568f9/d32bb895-5dd5-4c02-b031-f9ed3ff2fbb5"
-          (reference "#PWR019") (unit 1)
-        )
-        (path "/66d98af2-097e-4f68-99f2-351c9b9568f9/214ea90b-349a-415c-a8ca-f88377356f85"
-          (reference "#PWR027") (unit 1)
         )
       )
@@
           (reference "U2") (unit 4)
         )
-        (path "/66d98af2-097e-4f68-99f2-351c9b9568f9/d32bb895-5dd5-4c02-b031-f9ed3ff2fbb5"
-          (reference "U3") (unit 4)
-        )
-        (path "/66d98af2-097e-4f68-99f2-351c9b9568f9/214ea90b-349a-415c-a8ca-f88377356f85"
-          (reference "U4") (unit 4)
-        )
       )
     )
@@
         (path "/66d98af2-097e-4f68-99f2-351c9b9568f9/edbb582d-fe2b-48b6-8d6d-cfd6eb008018"
           (reference "#PWR02") (unit 1)
-        )
-        (path "/66d98af2-097e-4f68-99f2-351c9b9568f9/d32bb895-5dd5-4c02-b031-f9ed3ff2fbb5"
-          (reference "#PWR05") (unit 1)
-        )
-        (path "/66d98af2-097e-4f68-99f2-351c9b9568f9/214ea90b-349a-415c-a8ca-f88377356f85"
-          (reference "#PWR06") (unit 1)
         )
       )
@@
           (reference "U2") (unit 2)
         )
-        (path "/66d98af2-097e-4f68-99f2-351c9b9568f9/d32bb895-5dd5-4c02-b031-f9ed3ff2fbb5"
-          (reference "U3") (unit 2)
-        )
-        (path "/66d98af2-097e-4f68-99f2-351c9b9568f9/214ea90b-349a-415c-a8ca-f88377356f85"
-          (reference "U4") (unit 2)
-        )
       )
     )
@@
           (reference "#PWR016") (unit 1)
         )
-        (path "/66d98af2-097e-4f68-99f2-351c9b9568f9/d32bb895-5dd5-4c02-b031-f9ed3ff2fbb5"
-          (reference "#PWR024") (unit 1)
-        )
-        (path "/66d98af2-097e-4f68-99f2-351c9b9568f9/214ea90b-349a-415c-a8ca-f88377356f85"
-          (reference "#PWR032") (unit 1)
-        )
       )
     )
@@
         (path "/66d98af2-097e-4f68-99f2-351c9b9568f9/edbb582d-fe2b-48b6-8d6d-cfd6eb008018"
           (reference "#PWR012") (unit 1)
-        )
-        (path "/66d98af2-097e-4f68-99f2-351c9b9568f9/d32bb895-5dd5-4c02-b031-f9ed3ff2fbb5"
-          (reference "#PWR020") (unit 1)
-        )
-        (path "/66d98af2-097e-4f68-99f2-351c9b9568f9/214ea90b-349a-415c-a8ca-f88377356f85"
-          (reference "#PWR028") (unit 1)
         )
       )
@@
         (path "/66d98af2-097e-4f68-99f2-351c9b9568f9/edbb582d-fe2b-48b6-8d6d-cfd6eb008018"
           (reference "D5") (unit 1)
-        )
-        (path "/66d98af2-097e-4f68-99f2-351c9b9568f9/d32bb895-5dd5-4c02-b031-f9ed3ff2fbb5"
-          (reference "D9") (unit 1)
-        )
-        (path "/66d98af2-097e-4f68-99f2-351c9b9568f9/214ea90b-349a-415c-a8ca-f88377356f85"
-          (reference "D13") (unit 1)
         )
       )
@@
           (reference "U2") (unit 1)
         )
-        (path "/66d98af2-097e-4f68-99f2-351c9b9568f9/d32bb895-5dd5-4c02-b031-f9ed3ff2fbb5"
-          (reference "U3") (unit 1)
-        )
-        (path "/66d98af2-097e-4f68-99f2-351c9b9568f9/214ea90b-349a-415c-a8ca-f88377356f85"
-          (reference "U4") (unit 1)
-        )
       )
     )
@@
         (path "/66d98af2-097e-4f68-99f2-351c9b9568f9/edbb582d-fe2b-48b6-8d6d-cfd6eb008018"
           (reference "#PWR015") (unit 1)
-        )
-        (path "/66d98af2-097e-4f68-99f2-351c9b9568f9/d32bb895-5dd5-4c02-b031-f9ed3ff2fbb5"
-          (reference "#PWR023") (unit 1)
-        )
-        (path "/66d98af2-097e-4f68-99f2-351c9b9568f9/214ea90b-349a-415c-a8ca-f88377356f85"
-          (reference "#PWR031") (unit 1)
         )
       )
@@
           (reference "D7") (unit 1)
         )
-        (path "/66d98af2-097e-4f68-99f2-351c9b9568f9/d32bb895-5dd5-4c02-b031-f9ed3ff2fbb5"
-          (reference "D11") (unit 1)
-        )
-        (path "/66d98af2-097e-4f68-99f2-351c9b9568f9/214ea90b-349a-415c-a8ca-f88377356f85"
-          (reference "D15") (unit 1)
-        )
       )
     )
@@
         (path "/66d98af2-097e-4f68-99f2-351c9b9568f9/edbb582d-fe2b-48b6-8d6d-cfd6eb008018"
           (reference "#PWR018") (unit 1)
-        )
-        (path "/66d98af2-097e-4f68-99f2-351c9b9568f9/d32bb895-5dd5-4c02-b031-f9ed3ff2fbb5"
-          (reference "#PWR021") (unit 1)
-        )
-        (path "/66d98af2-097e-4f68-99f2-351c9b9568f9/214ea90b-349a-415c-a8ca-f88377356f85"
-          (reference "#PWR022") (unit 1)
         )
       )
@@
           (reference "U2") (unit 3)
         )
-        (path "/66d98af2-097e-4f68-99f2-351c9b9568f9/d32bb895-5dd5-4c02-b031-f9ed3ff2fbb5"
-          (reference "U3") (unit 3)
-        )
-        (path "/66d98af2-097e-4f68-99f2-351c9b9568f9/214ea90b-349a-415c-a8ca-f88377356f85"
-          (reference "U4") (unit 3)
-        )
       )
     )
@@
           (reference "D8") (unit 1)
         )
-        (path "/66d98af2-097e-4f68-99f2-351c9b9568f9/d32bb895-5dd5-4c02-b031-f9ed3ff2fbb5"
-          (reference "D12") (unit 1)
-        )
-        (path "/66d98af2-097e-4f68-99f2-351c9b9568f9/214ea90b-349a-415c-a8ca-f88377356f85"
-          (reference "D16") (unit 1)
-        )
       )
     )
@@
           (reference "D6") (unit 1)
         )
-        (path "/66d98af2-097e-4f68-99f2-351c9b9568f9/d32bb895-5dd5-4c02-b031-f9ed3ff2fbb5"
-          (reference "D10") (unit 1)
-        )
-        (path "/66d98af2-097e-4f68-99f2-351c9b9568f9/214ea90b-349a-415c-a8ca-f88377356f85"
-          (reference "D14") (unit 1)
-        )
       )
     )
@@
           (reference "#PWR026") (unit 1)
         )
-        (path "/66d98af2-097e-4f68-99f2-351c9b9568f9/d32bb895-5dd5-4c02-b031-f9ed3ff2fbb5"
-          (reference "#PWR029") (unit 1)
-        )
-        (path "/66d98af2-097e-4f68-99f2-351c9b9568f9/214ea90b-349a-415c-a8ca-f88377356f85"
-          (reference "#PWR030") (unit 1)
-        )
       )
     )
@@
           (reference "#PWR010") (unit 1)
         )
-        (path "/66d98af2-097e-4f68-99f2-351c9b9568f9/d32bb895-5dd5-4c02-b031-f9ed3ff2fbb5"
-          (reference "#PWR013") (unit 1)
-        )
-        (path "/66d98af2-097e-4f68-99f2-351c9b9568f9/214ea90b-349a-415c-a8ca-f88377356f85"
-          (reference "#PWR014") (unit 1)
-        )
-      )
+      )
