File: boards/rgb-input/rgb-input.kicad_sch (KiCad schematic)
At the start: 6 parts, among them J42 INPUTS, U1 ESP32-DEVKITC

Commit message: added 5v fuse to schematic
Changed lines of the file:
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@@
+    (stroke (width 0) (type default))
+  )
+  (wire (pts (xy 179.705 68.58) (xy 179.705 86.36))
     (stroke (width 0) (type default))
   )
@@
   )
   (wire (pts (xy 239.395 86.36) (xy 221.615 86.36))
-    (stroke (width 0) (type default))
-  )
-  (wire (pts (xy 179.705 81.28) (xy 179.705 86.36))
     (stroke (width 0) (type default))
   )
@@
     )
   )
-  (symbol (lib_id "power:+3.3V") (at 179.705 81.28 0) (unit 1)
+  (symbol (lib_id "power:+3.3V") (at 179.705 68.58 0) (unit 1)
     (in_bom yes) (on_board yes) (dnp no) (fields_autoplaced)
-    (property "Reference" "#PWR02" (at 179.705 85.09 0)
-      (effects (font (size 1.27 1.27)) hide)
-    )
-    (property "Value" "+3.3V" (at 179.705 76.2 0)
+    (property "Reference" "#PWR02" (at 179.705 72.39 0)
+      (effects (font (size 1.27 1.27)) hide)
+    )
+    (property "Value" "+3.3V" (at 179.705 63.5 0)
       (effects (font (size 1.27 1.27)))
     )
-    (property "Footprint" "" (at 179.705 81.28 0)
-      (effects (font (size 1.27 1.27)) hide)
-    )
-    (property "Datasheet" "" (at 179.705 81.28 0)
-      (effects (font (size 1.27 1.27)) hide)
-    )
+    (property "Footprint" "" (at 179.705 68.58 0)
+      (effects (font (size 1.27 1.27)) hide)
+    )
+    (property "Datasheet" "" (at 179.705 68.58 0)
+      (effects (font (size 1.27 1.27)) hide)
+    )

Commit message: rgb input board ready for production too.
Parts:
- U1: footprint gnarboard:ESP32-DevKitC -> yarrboard:ESP32-DevKitC
