File: boards/rgb-input/rgb-input.kicad_sch (KiCad schematic)
At the start: 6 parts, among them J42 INPUTS, U1 ESP32-DEVKITC

Commit message: more BOM updates.
Parts:
- H1, H2, H3, H4: now left out of the parts list
- J42: LCSC (none) -> C115249
- U1: Mouser (none) -> 356-ESP32-DEVKITC32E; Vendor 356-ESP32-DEVKITC32E -> (none)
Changed lines of the file:
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@@
   )
   (symbol (lib_id "Mechanical:MountingHole_Pad") (at 15.875 187.325 0) (unit 1)
-    (in_bom yes) (on_board yes) (dnp no) (fields_autoplaced)
+    (in_bom no) (on_board yes) (dnp no) (fields_autoplaced)
     (property "Reference" "H3" (at 18.415 186.055 0)
       (effects (font (size 1.27 1.27)) (justify left))
@@
   )
   (symbol (lib_id "Mechanical:MountingHole_Pad") (at 15.875 180.34 0) (unit 1)
-    (in_bom yes) (on_board yes) (dnp no) (fields_autoplaced)
+    (in_bom no) (on_board yes) (dnp no) (fields_autoplaced)
     (property "Reference" "H2" (at 18.415 179.07 0)
       (effects (font (size 1.27 1.27)) (justify left))
@@
       (effects (font (size 1.27 1.27)) hide)
     )
-    (property "Vendor" "356-ESP32-DEVKITC32E " (at 202.565 107.95 0)
+    (property "Mouser" "356-ESP32-DEVKITC32E " (at 202.565 107.95 0)
       (effects (font (size 1.27 1.27)) hide)
     )
@@
   )
   (symbol (lib_id "Mechanical:MountingHole_Pad") (at 15.875 173.355 0) (unit 1)
-    (in_bom yes) (on_board yes) (dnp no) (fields_autoplaced)
+    (in_bom no) (on_board yes) (dnp no) (fields_autoplaced)
     (property "Reference" "H1" (at 18.415 172.085 0)
       (effects (font (size 1.27 1.27)) (justify left))
@@
   )
   (symbol (lib_id "Mechanical:MountingHole_Pad") (at 15.875 194.31 0) (unit 1)
-    (in_bom yes) (on_board yes) (dnp no) (fields_autoplaced)
+    (in_bom no) (on_board yes) (dnp no) (fields_autoplaced)
     (property "Reference" "H4" (at 18.415 193.04 0)
       (effects (font (size 1.27 1.27)) (justify left))
@@
       (effects (font (size 1.27 1.27)) hide)
     )
+    (property "LCSC" "C115249" (at 227.33 36.83 0)
+      (effects (font (size 1.27 1.27)) hide)
+    )

Commit message: first pass on redesign of the rgb input board
Parts:
- added R17: 0R, Resistor_SMD:R_0805_2012Metric_Pad1.20x1.40mm_HandSolder, symbol Device:R_Small_US
Connections:
- net INPUT0: no longer U1.15 (GPIO13)
- net INPUT1: no longer U1.13 (GPIO12)
- net INPUT2: now also U1.8 (GPIO33); no longer U1.12 (GPIO14)
- net INPUT3: no longer U1.11 (GPIO27)
- net INPUT4: no longer U1.10 (GPIO26)
- net INPUT5: now also U1.5 (GPIO34); no longer U1.9 (GPIO25)
- net INPUT6: now also U1.4 (GPIO39); no longer U1.8 (GPIO33)
- net INPUT7: no longer U1.7 (GPIO32)
- net LED_SS: now also U1.11 (GPIO27); no longer U1.23 (GPIO15)
- net INPUT10: no longer names the net of J42.15 (Pin_15)
- net INPUT10: no longer U1.4 (GPIO39)
- net INPUT11: no longer names the net of J42.16 (Pin_16)
- net INPUT11: no longer U1.3 (GPIO36)
- net INPUT12: no longer names the net of U1.24 (GPIO2)
- net INPUT12: no longer J42.17 (Pin_17)
- net INPUT13: no longer names the net of J42.18 (Pin_18)
- net INPUT13: no longer U1.26 (GPIO4)
- net INPUT14: no longer names the net of U1.27 (GPIO16)
- net INPUT14: no longer J42.19 (Pin_19)
- net INPUT15: no longer names the net of U1.29 (GPIO5)
- net INPUT15: no longer J42.20 (Pin_20)
- net INPUT8: no longer names the net of J42.13 (Pin_13)
- net INPUT8: no longer U1.6 (GPIO35)
- net INPUT9: no longer names the net of J42.14 (Pin_14)
- net INPUT9: no longer U1.5 (GPIO34)
- net MISO renamed ADC_MISO
- net MOSI renamed ADC_MOSI
- net SCK renamed ADC_SCK
- net SDA renamed SCA
- new net: R17.1, U1.13 (GPIO12)
- new net Input Switch0/INPUT: U1.10 (GPIO26)
- new net Input Switch1/INPUT: U1.9 (GPIO25)
- new net Input Switch3/INPUT: U1.7 (GPIO32)
- new net Input Switch4/INPUT: U1.6 (GPIO35)
- new net Input Switch7/INPUT: U1.3 (GPIO36)
- new net LED_BLANK: U1.26 (GPIO4)
- new net LED_MISO: R17.2
- new net LED_MOSI: U1.15 (GPIO13)
- new net LED_SCK: U1.12 (GPIO14)
- no-connect marks 14 -> 18
Other:
- removed sheet Input Switch10
- removed sheet Input Switch11
- removed sheet Input Switch12
- removed sheet Input Switch13
- removed sheet Input Switch14
- removed sheet Input Switch15
- removed sheet Input Switch8
- removed sheet Input Switch9
- moved on the sheet: U1

Commit message: new rgb input board coming along very nicely
Parts:
- J42: footprint Connector_IDC:IDC-Header_2x10_P2.54mm_Vertical -> Connector_FFC-FPC:Molex_200528-0100_1x10-1MP_P1.00mm_Horizontal; symbol Connector_Generic:Conn_02x10_Odd_Even -> Connector_Generic:Conn_01x10
Connections:
- net Input Switch0/INPUT is gone; now on net INPUT0: U1.10 (GPIO26)
- net Input Switch1/INPUT is gone; now on net INPUT1: U1.9 (GPIO25)
- net Input Switch3/INPUT is gone; now on net INPUT3: U1.7 (GPIO32)
- net Input Switch4/INPUT is gone; now on net INPUT4: U1.6 (GPIO35)
- net Input Switch7/INPUT is gone; now on net INPUT7: U1.3 (GPIO36)
- net +3.3V: no longer J42.3 (Pin_3)
- net GNDD: no longer J42.4 (Pin_4)
- net INPUT0: now also J42.3 (Pin_3); no longer J42.5 (Pin_5)
- net INPUT1: now also J42.4 (Pin_4); no longer J42.6 (Pin_6)
- net INPUT2: now also J42.5 (Pin_5); no longer J42.7 (Pin_7)
- net INPUT3: now also J42.6 (Pin_6); no longer J42.8 (Pin_8)
- net INPUT4: now also J42.7 (Pin_7); no longer J42.9 (Pin_9)
- net INPUT5: now also J42.8 (Pin_8); no longer J42.10 (Pin_10)
- net INPUT6: now also J42.9 (Pin_9); no longer J42.11 (Pin_11)
- net INPUT7: now also J42.10 (Pin_10); no longer J42.12 (Pin_12)

Commit message: new rgb input board is starting to look very nice.
Parts:
- J42: footprint Connector_FFC-FPC:Molex_200528-0100_1x10-1MP_P1.00mm_Horizontal -> Connector_FFC-FPC:TE_1-84952-0_1x10-1MP_P1.0mm_Horizontal; LCSC C115249 -> C262385
Connections:
- net SCA renamed SDA
Changed lines of the file:
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@@
     )
   )
-  (global_label "SCA" (shape input) (at 223.52 99.06 0) (fields_autoplaced)
+  (global_label "SDA" (shape input) (at 223.52 99.06 0) (fields_autoplaced)
     (effects (font (size 1.27 1.27)) (justify left))
     (property "Intersheetrefs" "${INTERSHEET_REFS}" (at 230.0733 99.06 0)
@@
       (effects (font (size 1.27 1.27)) (justify left))
     )
-    (property "Footprint" "Connector_FFC-FPC:Molex_200528-0100_1x10-1MP_P1.00mm_Horizontal" (at 227.33 36.83 0)
+    (property "Footprint" "Connector_FFC-FPC:TE_1-84952-0_1x10-1MP_P1.0mm_Horizontal" (at 227.33 36.83 0)
       (effects (font (size 1.27 1.27)) hide)
     )
@@
       (effects (font (size 1.27 1.27)) hide)
     )
-    (property "LCSC" "C115249" (at 227.33 36.83 0)
-      (effects (font (size 1.27 1.27)) hide)
-    )
+    (property "LCSC" "C262385" (at 227.33 36.83 0)
+      (effects (font (size 1.27 1.27)) hide)
+    )

Commit message: passing ERC and DRC
Parts:
- J42: symbol Connector_Generic:Conn_01x10 -> Connector_Generic_MountingPin:Conn_01x10_MountingPin
- U1: symbol gnarboard:ESP32_DevKit_C -> yarrboard:ESP32_DevKit_C
Connections:
- net GNDD: now also J42.MP (MountPin)
Other:
- moved on the sheet: H1, H2, H3, H4

Commit message: reannotated and did some more cleanup.  almost ready
Parts:
- renumbered J42 to J1, R17 to R1
Connections:
- net GNDD: now also H1.1, H2.1, H3.1, H4.1
- no-connect marks 18 -> 14
Other:
- company: (none) -> github.com/hoeken/yarrboard
- title: (none) -> RGB Input Board
- moved on the sheet: H1, H2, H3, H4

Commit message: parts list updated
Parts:
- J1: LCSC C262385 -> C262385 or C52162; Manufacturer (none) -> AFA07-S10FCC-00 or AFA01-S10FCC-00
Changed lines of the file:
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@@
       (effects (font (size 1.27 1.27)) hide)
     )
-    (property "LCSC" "C262385" (at 54.61 53.34 0)
+    (property "LCSC" "C262385 or C52162" (at 54.61 53.34 0)
       (effects (font (size 1.27 1.27)) hide)
     )
+    (property "Manufacturer" "AFA07-S10FCC-00 or AFA01-S10FCC-00" (at 54.61 53.34 0)
+      (effects (font (size 1.27 1.27)) hide)
+    )
