File: boards/rgb-input/power.kicad_sch (KiCad schematic)
At the start: 19 parts, among them J1 Barrel_Jack, U3 XL1509-5.0

Commit message: more BOM updates.
Parts:
- C1, C2: Vendor 08053C104KAT4A -> (none)
- C1: LCSC (none) -> C90975; Vendor TAJC107K010RNJ -> (none)
- D26: LCSC (none) -> C908229; Mouser (none) -> 610-CMHSH5-2L; Vendor 610-CMHSH5-2L -> (none)
- D26: Mouser (none) -> 241-SX33L_R1_00001; Vendor 610-CMHSH5-2L -> (none)
- D31: value PESD5V0L1BA -> SMBJ30CA; footprint Diode_SMD:D_SOD-323_HandSoldering -> Diode_SMD:D_SMB; LCSC (none) -> C284101
- F1: value mSMD100 -> mSMD110; LCSC (none) -> C69691
- F9: LCSC (none) -> C70113
- FB4: LCSC (none) -> C1017
- J1: footprint Connector_BarrelJack:BarrelJack_CUI_PJ-063AH_Horizontal -> Connector_BarrelJack:BarrelJack_Horizontal; symbol Connector:Barrel_Jack_MountingPin -> Connector:Barrel_Jack; LCSC (none) -> C431533
- L1: LCSC (none) -> C90321
- L2: LCSC (none) -> C2894721
- R38: Vendor 652-CR0805JW-102ELF -> (none)
- U3: LCSC (none) -> C2902368
Connections:
- net GNDD: no longer J1.MP (MountPin)
Changed lines of the file:
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@@
   (junction (at 31.75 87.63) (diameter 0) (color 0 0 0 0)
   )
-  (junction (at 31.75 97.79) (diameter 0) (color 0 0 0 0)
-  )
   (junction (at 31.75 80.01) (diameter 0) (color 0 0 0 0)
   )
@@
   )
   (wire (pts (xy 222.25 80.01) (xy 231.14 80.01))
-    (stroke (width 0) (type default))
-  )
-  (wire (pts (xy 22.86 97.79) (xy 31.75 97.79))
     (stroke (width 0) (type default))
   )
@@
       (effects (font (size 1.27 1.27)) hide)
     )
-    (property "Vendor" "08053C104KAT4A" (at 149.86 87.63 0)
-      (effects (font (size 1.27 1.27)) hide)
-    )
     (pin "1")
     (pin "2")
@@
       (effects (font (size 1.27 1.27)) hide)
     )
-    (property "Vendor" " 610-CMHSH5-2L" (at 189.23 91.44 90)
+    (property "Mouser" " 610-CMHSH5-2L " (at 189.23 91.44 90)
+      (effects (font (size 1.27 1.27)) hide)
+    )
+    (property "LCSC" "C908229" (at 189.23 91.44 90)
       (effects (font (size 1.27 1.27)) hide)
     )
@@
       (effects (font (size 1.27 1.27)) hide)
     )
-    (property "Vendor" " 610-CMHSH5-2L" (at 242.57 80.01 90)
+    (property "Mouser" " 241-SX33L_R1_00001" (at 242.57 80.01 90)
       (effects (font (size 1.27 1.27)) hide)
     )
@@
       (effects (font (size 1.27 1.27)) hide)
     )
+    (property "LCSC" "C2894721" (at 201.93 80.01 90)
+      (effects (font (size 1.27 1.27)) hide)
+    )
     (pin "1")
     (pin "2")
@@
       (effects (font (size 1.27 1.27)) hide)
     )
-    (property "Vendor" "08053C104KAT4A" (at 120.65 87.63 0)
-      (effects (font (size 1.27 1.27)) hide)
-    )
     (pin "1")
     (pin "2")
@@
       (effects (font (size 1.27 1.27)) hide)
     )
+    (property "LCSC" "C90321" (at 110.49 80.01 90)
+      (effects (font (size 1.27 1.27)) hide)
+    )
     (pin "1")
     (pin "2")
@@
       (effects (font (size 1.27 1.27)) hide)
     )
-    (property "Vendor" "TAJC107K010RNJ" (at 231.14 87.63 0)
+    (property "LCSC" "C90975" (at 231.14 87.63 0)
       (effects (font (size 1.27 1.27)) hide)
     )
@@
       (effects (font (size 1.27 1.27)) (justify right))
     )
-    (property "Value" "PESD5V0L1BA" (at 88.9 88.9 90)
+    (property "Value" "SMBJ30CA" (at 88.9 88.9 90)
       (effects (font (size 1.27 1.27)) (justify right))
     )
-    (property "Footprint" "Diode_SMD:D_SOD-323_HandSoldering" (at 86.36 87.63 0)
+    (property "Footprint" "Diode_SMD:D_SMB" (at 86.36 87.63 0)
       (effects (font (size 1.27 1.27)) hide)
     )
     (property "Datasheet" "~" (at 86.36 87.63 0)
+      (effects (font (size 1.27 1.27)) hide)
+    )
+    (property "LCSC" "C284101" (at 86.36 87.63 90)
       (effects (font (size 1.27 1.27)) hide)
     )
@@
       (effects (font (size 1.27 1.27)) hide)
     )
+    (property "LCSC" "C1017" (at 55.88 80.01 90)
+      (effects (font (size 1.27 1.27)) hide)
+    )
     (pin "1")
     (pin "2")
@@
       (effects (font (size 1.27 1.27)))
     )
-    (property "Value" "mSMD100" (at 219.71 76.2 90)
+    (property "Value" "mSMD110" (at 219.71 76.2 90)
       (effects (font (size 1.27 1.27)))
     )
@@
       (effects (font (size 1.27 1.27)) hide)
     )
+    (property "LCSC" "C69691" (at 219.71 80.01 90)
+      (effects (font (size 1.27 1.27)) hide)
+    )
     (pin "1")
     (pin "2")
@@
     )
   )
-  (symbol (lib_id "Connector:Barrel_Jack_MountingPin") (at 22.86 90.17 0) (unit 1)
+  (symbol (lib_id "Connector:Barrel_Jack") (at 22.86 90.17 0) (unit 1)
     (in_bom yes) (on_board yes) (dnp no) (fields_autoplaced)
     (property "Reference" "J1" (at 22.86 81.28 0)
@@
       (effects (font (size 1.27 1.27)))
     )
-    (property "Footprint" "Connector_BarrelJack:BarrelJack_CUI_PJ-063AH_Horizontal" (at 24.13 91.186 0)
+    (property "Footprint" "Connector_BarrelJack:BarrelJack_Horizontal" (at 24.13 91.186 0)
       (effects (font (size 1.27 1.27)) hide)
     )
@@
       (effects (font (size 1.27 1.27)) hide)
     )
-    (pin "1")
-    (pin "2")
-    (pin "MP")
+    (property "LCSC" "C431533" (at 22.86 90.17 0)
+      (effects (font (size 1.27 1.27)) hide)
+    )
+    (pin "1")
+    (pin "2")
     (instances
       (project "rgb-input"
@@
       (effects (font (size 1.27 1.27)) hide)
     )
-    (property "Vendor" "08053C104KAT4A" (at 69.85 87.63 0)
-      (effects (font (size 1.27 1.27)) hide)
-    )
     (pin "1")
     (pin "2")
@@
       (effects (font (size 1.27 1.27)) hide)
     )
-    (property "Vendor" "08053C104KAT4A" (at 134.62 83.82 0)
-      (effects (font (size 1.27 1.27)) hide)
-    )
     (pin "1")
     (pin "2")
@@
     )
     (property "Datasheet" "~" (at 134.62 91.44 0)
-      (effects (font (size 1.27 1.27)) hide)
-    )
-    (property "Vendor" " 652-CR0805JW-102ELF " (at 134.62 91.44 0)
       (effects (font (size 1.27 1.27)) hide)
     )
@@
       (effects (font (size 1.27 1.27)) hide)
     )
+    (property "LCSC" "C70113" (at 40.64 80.01 90)
+      (effects (font (size 1.27 1.27)) hide)
+    )
     (pin "1")
     (pin "2")
@@
     )
     (property "Datasheet" "https://datasheet.lcsc.com/lcsc/1809050422_XLSEMI-XL1509-5-0E1_C61063.pdf" (at 176.53 71.882 0)
+      (effects (font (size 1.27 1.27)) hide)
+    )
+    (property "LCSC" "C2902368" (at 173.99 82.55 0)
       (effects (font (size 1.27 1.27)) hide)
     )
@@
       (effects (font (size 1.27 1.27)) hide)
     )
-    (property "Vendor" " 652-CR0805JW-102ELF " (at 184.15 111.76 0)
-      (effects (font (size 1.27 1.27)) hide)
-    )
     (pin "1")
     (pin "2")
@@
       (effects (font (size 1.27 1.27)) hide)
     )
-    (property "Vendor" " 610-CMHSH5-2L" (at 95.25 80.01 90)
-      (effects (font (size 1.27 1.27)) hide)
-    )
+    (property "Mouser" " 241-SX33L_R1_00001" (at 95.25 80.01 90)
+      (effects (font (size 1.27 1.27)) hide)
+    )

Commit message: updated inductor footprint
Parts:
- L2: footprint Inductor_SMD:L_Chilisin_BMRA00040420 -> Inductor_SMD:L_Chilisin_BMRB00060650
Changed lines of the file:
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@@
       (effects (font (size 1.27 1.27)))
     )
-    (property "Footprint" "Inductor_SMD:L_Chilisin_BMRA00040420" (at 201.93 80.01 0)
+    (property "Footprint" "Inductor_SMD:L_Chilisin_BMRB00060650" (at 201.93 80.01 0)
       (effects (font (size 1.27 1.27)) hide)
     )
