File: boards/rgb-input/adc input.kicad_sch (KiCad schematic)
At the start: 4 parts

Commit message: new rgb input board is starting to look very nice.
Parts:
- renumbered C11 to C19
Changed lines of the file:
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@@
   (symbol (lib_id "Device:C_Small") (at 162.56 96.52 0) (unit 1)
     (in_bom yes) (on_board yes) (dnp no) (fields_autoplaced)
-    (property "Reference" "C11" (at 165.1 95.2563 0)
+    (property "Reference" "C19" (at 165.1 95.2563 0)
       (effects (font (size 1.27 1.27)) (justify left))
     )

Commit message: reannotated and did some more cleanup.  almost ready
Parts:
- renumbered C19 to C22, D12 to D13, R19 to R21
Other:
- company: (none) -> github.com/hoeken/yarrboard
- title: (none) -> RGB Input Board
