File: boards/rgb-input/input switch.kicad_sch (KiCad schematic)
At the start: 5 parts

Commit message: passing ERC and DRC
Other:
- moved on the sheet: C3, D2, INPUT0, R1, R2

Commit message: reannotated and did some more cleanup.  almost ready
Parts:
- renumbered C3 to C4, D2 to D7, R2 to R10, R1 to R11
Other:
- company: (none) -> github.com/hoeken/yarrboard
- title: (none) -> RGB Input Board
