File: boards/rgb-input/led driver.kicad_sch (KiCad schematic)
At the start: 4 parts, among them U6 TLC5947DAP

Commit message: more BOM updates.
Parts:
- U6: Mouser (none) -> 595-TLC5947DAPR
Changed lines of the file:
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@@
+      (effects (font (size 1.27 1.27)) hide)
+    )
+    (property "Mouser" " 595-TLC5947DAPR " (at 116.84 91.44 0)
       (effects (font (size 1.27 1.27)) hide)
     )

Commit message: updated inductor footprint
Parts:
- renumbered C23 to C3, R13 to R1

Commit message: solved the ADC issue and found another minor one
Parts:
- renumbered C3 to C23, R1 to R20

Commit message: first pass on redesign of the rgb input board
Parts:
- renumbered C23 to C3, R20 to R13

Commit message: new rgb input board coming along very nicely
Parts:
- removed R13: 10k, Resistor_SMD:R_0805_2012Metric, symbol Device:R_US
- renumbered R13 to R20
Changed lines of the file:
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@@
   (junction (at 121.92 52.07) (diameter 0) (color 0 0 0 0)
   )
-  (junction (at 84.455 76.2) (diameter 0) (color 0 0 0 0)
-  )
-  (junction (at 84.455 86.36) (diameter 0) (color 0 0 0 0)
-  )
   (junction (at 119.38 128.905) (diameter 0) (color 0 0 0 0)
   )
@@
     (stroke (width 0) (type default))
   )
-  (wire (pts (xy 84.455 76.2) (xy 72.39 76.2))
-    (stroke (width 0) (type default))
-  )
-  (wire (pts (xy 84.455 83.82) (xy 84.455 86.36))
-    (stroke (width 0) (type default))
-  )
   (wire (pts (xy 114.3 128.905) (xy 116.84 128.905))
     (stroke (width 0) (type default))
   )
-  (wire (pts (xy 84.455 86.36) (xy 99.06 86.36))
-    (stroke (width 0) (type default))
-  )
   (wire (pts (xy 114.3 128.905) (xy 114.3 127))
     (stroke (width 0) (type default))
@@
     (stroke (width 0) (type default))
   )
-  (wire (pts (xy 70.485 86.36) (xy 84.455 86.36))
+  (wire (pts (xy 70.485 86.36) (xy 99.06 86.36))
     (stroke (width 0) (type default))
   )
@@
     (stroke (width 0) (type default))
   )
-  (wire (pts (xy 95.25 76.2) (xy 84.455 76.2))
+  (wire (pts (xy 72.39 76.2) (xy 95.25 76.2))
     (stroke (width 0) (type default))
   )
@@
   (symbol (lib_id "Device:R_US") (at 95.25 80.01 0) (mirror x) (unit 1)
     (in_bom yes) (on_board yes) (dnp no) (fields_autoplaced)
-    (property "Reference" "R13" (at 92.71 78.74 0)
+    (property "Reference" "R20" (at 92.71 78.74 0)
       (effects (font (size 1.27 1.27)) (justify right))
     )
@@
     (instances
       (project "rgb-input"
+        (path "/c83c6236-96e9-46ad-9d7a-9e2efa4a7966/120468c6-3bec-414c-9049-57af589f397a"
+          (reference "R20") (unit 1)
+        )
+        (path "/c83c6236-96e9-46ad-9d7a-9e2efa4a7966/4f50afed-9381-4977-8e27-209f0f88ad4e"
+          (reference "R3") (unit 1)
+        )
+        (path "/c83c6236-96e9-46ad-9d7a-9e2efa4a7966/4175a172-5c0b-4d6a-88bb-129f5f07b813"
+          (reference "R5") (unit 1)
+        )
+        (path "/c83c6236-96e9-46ad-9d7a-9e2efa4a7966/6f6f2d8d-82f6-4691-bba7-8caa1bd52e96"
+          (reference "R7") (unit 1)
+        )
+        (path "/c83c6236-96e9-46ad-9d7a-9e2efa4a7966/145fa34f-e19e-43e2-bb48-aff2e824ef0a"
+          (reference "R9") (unit 1)
+        )
+        (path "/c83c6236-96e9-46ad-9d7a-9e2efa4a7966/5fc618b8-7830-4bbf-bf46-7753631e9b1e"
+          (reference "R11") (unit 1)
+        )
+        (path "/c83c6236-96e9-46ad-9d7a-9e2efa4a7966/f06c9bf0-de4e-49a2-91ec-1c9426377826"
+          (reference "R19") (unit 1)
+        )
+        (path "/c83c6236-96e9-46ad-9d7a-9e2efa4a7966/803edf1a-5825-4947-a8b9-85d3a29697e5"
+          (reference "R15") (unit 1)
+        )
         (path "/c83c6236-96e9-46ad-9d7a-9e2efa4a7966/802175d5-fb4b-4457-a117-b0f397189ff7"
           (reference "R13") (unit 1)
         )
-        (path "/c83c6236-96e9-46ad-9d7a-9e2efa4a7966/4f50afed-9381-4977-8e27-209f0f88ad4e"
-          (reference "R3") (unit 1)
-        )
-        (path "/c83c6236-96e9-46ad-9d7a-9e2efa4a7966/4175a172-5c0b-4d6a-88bb-129f5f07b813"
-          (reference "R5") (unit 1)
-        )
-        (path "/c83c6236-96e9-46ad-9d7a-9e2efa4a7966/6f6f2d8d-82f6-4691-bba7-8caa1bd52e96"
-          (reference "R7") (unit 1)
-        )
-        (path "/c83c6236-96e9-46ad-9d7a-9e2efa4a7966/145fa34f-e19e-43e2-bb48-aff2e824ef0a"
-          (reference "R9") (unit 1)
-        )
-        (path "/c83c6236-96e9-46ad-9d7a-9e2efa4a7966/5fc618b8-7830-4bbf-bf46-7753631e9b1e"
-          (reference "R11") (unit 1)
-        )
-        (path "/c83c6236-96e9-46ad-9d7a-9e2efa4a7966/f06c9bf0-de4e-49a2-91ec-1c9426377826"
-          (reference "R19") (unit 1)
-        )
-        (path "/c83c6236-96e9-46ad-9d7a-9e2efa4a7966/803edf1a-5825-4947-a8b9-85d3a29697e5"
-          (reference "R15") (unit 1)
-        )
         (path "/c83c6236-96e9-46ad-9d7a-9e2efa4a7966/ef548cdc-9d5d-4f8e-8f54-0c2e96dbe3f0"
           (reference "R1") (unit 1)
-        )
-        (path "/c83c6236-96e9-46ad-9d7a-9e2efa4a7966/120468c6-3bec-414c-9049-57af589f397a"
-          (reference "R20") (unit 1)
         )
         (path "/c83c6236-96e9-46ad-9d7a-9e2efa4a7966/c9e1b2da-9064-45a5-a0a2-ee072f7e1acf"
@@
         )
       )
-    )
-  )
-  (symbol (lib_id "Device:R_US") (at 84.455 80.01 0) (mirror x) (unit 1)
-    (in_bom yes) (on_board yes) (dnp no) (fields_autoplaced)
-    (property "Reference" "R13" (at 81.915 78.74 0)
-      (effects (font (size 1.27 1.27)) (justify right))
-    )
-    (property "Value" "10k" (at 81.915 81.28 0)
-      (effects (font (size 1.27 1.27)) (justify right))
-    )
-    (property "Footprint" "Resistor_SMD:R_0805_2012Metric" (at 85.471 79.756 90)
-      (effects (font (size 1.27 1.27)) hide)
-    )
-    (property "Datasheet" "~" (at 84.455 80.01 0)
-      (effects (font (size 1.27 1.27)) hide)
-    )
-    (pin "1")
-    (pin "2")
-    (instances
-      (project "rgb-input"
-        (path "/c83c6236-96e9-46ad-9d7a-9e2efa4a7966/802175d5-fb4b-4457-a117-b0f397189ff7"
-          (reference "R13") (unit 1)
-        )
-        (path "/c83c6236-96e9-46ad-9d7a-9e2efa4a7966/4f50afed-9381-4977-8e27-209f0f88ad4e"
-          (reference "R3") (unit 1)
-        )
-        (path "/c83c6236-96e9-46ad-9d7a-9e2efa4a7966/4175a172-5c0b-4d6a-88bb-129f5f07b813"
-          (reference "R5") (unit 1)
-        )
-        (path "/c83c6236-96e9-46ad-9d7a-9e2efa4a7966/6f6f2d8d-82f6-4691-bba7-8caa1bd52e96"
-          (reference "R7") (unit 1)
-        )
-        (path "/c83c6236-96e9-46ad-9d7a-9e2efa4a7966/145fa34f-e19e-43e2-bb48-aff2e824ef0a"
-          (reference "R9") (unit 1)
-        )
-        (path "/c83c6236-96e9-46ad-9d7a-9e2efa4a7966/5fc618b8-7830-4bbf-bf46-7753631e9b1e"
-          (reference "R11") (unit 1)
-        )
-        (path "/c83c6236-96e9-46ad-9d7a-9e2efa4a7966/f06c9bf0-de4e-49a2-91ec-1c9426377826"
-          (reference "R19") (unit 1)
-        )
-        (path "/c83c6236-96e9-46ad-9d7a-9e2efa4a7966/803edf1a-5825-4947-a8b9-85d3a29697e5"
-          (reference "R15") (unit 1)
-        )
-        (path "/c83c6236-96e9-46ad-9d7a-9e2efa4a7966/ef548cdc-9d5d-4f8e-8f54-0c2e96dbe3f0"
-          (reference "R1") (unit 1)
-        )
-        (path "/c83c6236-96e9-46ad-9d7a-9e2efa4a7966/120468c6-3bec-414c-9049-57af589f397a"
-          (reference "R20") (unit 1)
-        )
-        (path "/c83c6236-96e9-46ad-9d7a-9e2efa4a7966/c9e1b2da-9064-45a5-a0a2-ee072f7e1acf"
-          (reference "R21") (unit 1)
-        )
-        (path "/c83c6236-96e9-46ad-9d7a-9e2efa4a7966/1ca70e91-4481-4c96-8c08-39dd142498e5"
-          (reference "R22") (unit 1)
-        )
-        (path "/c83c6236-96e9-46ad-9d7a-9e2efa4a7966/597c781a-3a73-4808-b6ed-8c917478e623"
-          (reference "R23") (unit 1)
-        )
-        (path "/c83c6236-96e9-46ad-9d7a-9e2efa4a7966/7fda9512-7a31-4b6e-85db-2478bfe7f375"
-          (reference "R24") (unit 1)
-        )
-        (path "/c83c6236-96e9-46ad-9d7a-9e2efa4a7966/d24c7443-0875-4d8e-b56e-81b211cd6f3d"
-          (reference "R25") (unit 1)
-        )
-        (path "/c83c6236-96e9-46ad-9d7a-9e2efa4a7966/76149826-8526-4a6c-8e11-6dc0109cc281"
-          (reference "R26") (unit 1)
-        )
-        (path "/c83c6236-96e9-46ad-9d7a-9e2efa4a7966/846833bc-7ec6-4ec6-86e7-310fef01b65c/720a8c4a-525c-4eec-8216-6ac4d044fce4"
-          (reference "R47") (unit 1)
-        )
-      )

Commit message: passing ERC and DRC
Parts:
- renumbered R20 to R1
Changed lines of the file:
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@@
   (junction (at 121.92 52.07) (diameter 0) (color 0 0 0 0)
   )
-  (junction (at 119.38 128.905) (diameter 0) (color 0 0 0 0)
-  )
-  (junction (at 116.84 128.905) (diameter 0) (color 0 0 0 0)
-  )
-  (wire (pts (xy 70.485 96.52) (xy 99.06 96.52))
-    (stroke (width 0) (type default))
-  )
-  (wire (pts (xy 119.38 128.905) (xy 119.38 127))
+  (junction (at 119.38 129.54) (diameter 0) (color 0 0 0 0)
+  )
+  (junction (at 116.84 129.54) (diameter 0) (color 0 0 0 0)
+  )
+  (wire (pts (xy 71.12 96.52) (xy 99.06 96.52))
+    (stroke (width 0) (type default))
+  )
+  (wire (pts (xy 119.38 127) (xy 119.38 129.54))
     (stroke (width 0) (type default))
   )
@@
     (stroke (width 0) (type default))
   )
-  (wire (pts (xy 70.485 88.9) (xy 99.06 88.9))
+  (wire (pts (xy 114.3 127) (xy 114.3 129.54))
+    (stroke (width 0) (type default))
+  )
+  (wire (pts (xy 71.12 88.9) (xy 99.06 88.9))
     (stroke (width 0) (type default))
   )
@@
     (stroke (width 0) (type default))
   )
-  (wire (pts (xy 70.485 93.98) (xy 99.06 93.98))
-    (stroke (width 0) (type default))
-  )
-  (wire (pts (xy 116.84 128.905) (xy 116.84 130.81))
-    (stroke (width 0) (type default))
-  )
-  (wire (pts (xy 114.3 128.905) (xy 116.84 128.905))
-    (stroke (width 0) (type default))
-  )
-  (wire (pts (xy 114.3 128.905) (xy 114.3 127))
+  (wire (pts (xy 71.12 93.98) (xy 99.06 93.98))
+    (stroke (width 0) (type default))
+  )
+  (wire (pts (xy 116.84 129.54) (xy 116.84 132.08))
+    (stroke (width 0) (type default))
+  )
+  (wire (pts (xy 114.3 129.54) (xy 116.84 129.54))
     (stroke (width 0) (type default))
   )
@@
     (stroke (width 0) (type default))
   )
-  (wire (pts (xy 70.485 86.36) (xy 99.06 86.36))
-    (stroke (width 0) (type default))
-  )
-  (wire (pts (xy 154.94 88.9) (xy 154.94 128.905))
+  (wire (pts (xy 71.12 86.36) (xy 99.06 86.36))
+    (stroke (width 0) (type default))
+  )
+  (wire (pts (xy 154.94 88.9) (xy 154.94 129.54))
     (stroke (width 0) (type default))
   )
@@
     (stroke (width 0) (type default))
   )
-  (wire (pts (xy 154.94 128.905) (xy 119.38 128.905))
-    (stroke (width 0) (type default))
-  )
-  (wire (pts (xy 70.485 91.44) (xy 99.06 91.44))
+  (wire (pts (xy 154.94 129.54) (xy 119.38 129.54))
+    (stroke (width 0) (type default))
+  )
+  (wire (pts (xy 71.12 91.44) (xy 99.06 91.44))
     (stroke (width 0) (type default))
   )
@@
     (stroke (width 0) (type default))
   )
-  (wire (pts (xy 119.38 128.905) (xy 116.84 128.905))
+  (wire (pts (xy 119.38 129.54) (xy 116.84 129.54))
     (stroke (width 0) (type default))
   )
@@
     (effects (font (size 1.27 1.27)) (justify left))
   )
-  (hierarchical_label "SIN" (shape input) (at 70.485 93.98 180) (fields_autoplaced)
+  (hierarchical_label "SIN" (shape input) (at 71.12 93.98 180) (fields_autoplaced)
     (effects (font (size 1.27 1.27)) (justify right))
   )
@@
     (effects (font (size 1.27 1.27)) (justify left))
   )
-  (hierarchical_label "XLAT" (shape input) (at 70.485 88.9 180) (fields_autoplaced)
-    (effects (font (size 1.27 1.27)) (justify right))
-  )
-  (hierarchical_label "SOUT" (shape input) (at 70.485 96.52 180) (fields_autoplaced)
+  (hierarchical_label "XLAT" (shape input) (at 71.12 88.9 180) (fields_autoplaced)
+    (effects (font (size 1.27 1.27)) (justify right))
+  )
+  (hierarchical_label "SOUT" (shape input) (at 71.12 96.52 180) (fields_autoplaced)
     (effects (font (size 1.27 1.27)) (justify right))
   )
@@
     (effects (font (size 1.27 1.27)) (justify left))
   )
-  (hierarchical_label "SCLK" (shape input) (at 70.485 91.44 180) (fields_autoplaced)
+  (hierarchical_label "SCLK" (shape input) (at 71.12 91.44 180) (fields_autoplaced)
     (effects (font (size 1.27 1.27)) (justify right))
   )
@@
     (effects (font (size 1.27 1.27)) (justify left))
   )
-  (hierarchical_label "BLANK" (shape input) (at 70.485 86.36 180) (fields_autoplaced)
+  (hierarchical_label "BLANK" (shape input) (at 71.12 86.36 180) (fields_autoplaced)
     (effects (font (size 1.27 1.27)) (justify right))
   )
@@
   (symbol (lib_id "Device:R_US") (at 95.25 80.01 0) (mirror x) (unit 1)
     (in_bom yes) (on_board yes) (dnp no) (fields_autoplaced)
-    (property "Reference" "R20" (at 92.71 78.74 0)
+    (property "Reference" "R1" (at 92.71 78.74 0)
       (effects (font (size 1.27 1.27)) (justify right))
     )
@@
     (instances
       (project "rgb-input"
+        (path "/c83c6236-96e9-46ad-9d7a-9e2efa4a7966/ef548cdc-9d5d-4f8e-8f54-0c2e96dbe3f0"
+          (reference "R1") (unit 1)
+        )
+        (path "/c83c6236-96e9-46ad-9d7a-9e2efa4a7966/4f50afed-9381-4977-8e27-209f0f88ad4e"
+          (reference "R3") (unit 1)
+        )
+        (path "/c83c6236-96e9-46ad-9d7a-9e2efa4a7966/4175a172-5c0b-4d6a-88bb-129f5f07b813"
+          (reference "R5") (unit 1)
+        )
+        (path "/c83c6236-96e9-46ad-9d7a-9e2efa4a7966/6f6f2d8d-82f6-4691-bba7-8caa1bd52e96"
+          (reference "R7") (unit 1)
+        )
+        (path "/c83c6236-96e9-46ad-9d7a-9e2efa4a7966/145fa34f-e19e-43e2-bb48-aff2e824ef0a"
+          (reference "R9") (unit 1)
+        )
+        (path "/c83c6236-96e9-46ad-9d7a-9e2efa4a7966/5fc618b8-7830-4bbf-bf46-7753631e9b1e"
+          (reference "R11") (unit 1)
+        )
+        (path "/c83c6236-96e9-46ad-9d7a-9e2efa4a7966/f06c9bf0-de4e-49a2-91ec-1c9426377826"
+          (reference "R19") (unit 1)
+        )
+        (path "/c83c6236-96e9-46ad-9d7a-9e2efa4a7966/803edf1a-5825-4947-a8b9-85d3a29697e5"
+          (reference "R15") (unit 1)
+        )
         (path "/c83c6236-96e9-46ad-9d7a-9e2efa4a7966/120468c6-3bec-414c-9049-57af589f397a"
           (reference "R20") (unit 1)
         )
-        (path "/c83c6236-96e9-46ad-9d7a-9e2efa4a7966/4f50afed-9381-4977-8e27-209f0f88ad4e"
-          (reference "R3") (unit 1)
-        )
-        (path "/c83c6236-96e9-46ad-9d7a-9e2efa4a7966/4175a172-5c0b-4d6a-88bb-129f5f07b813"
-          (reference "R5") (unit 1)
-        )
-        (path "/c83c6236-96e9-46ad-9d7a-9e2efa4a7966/6f6f2d8d-82f6-4691-bba7-8caa1bd52e96"
-          (reference "R7") (unit 1)
-        )
-        (path "/c83c6236-96e9-46ad-9d7a-9e2efa4a7966/145fa34f-e19e-43e2-bb48-aff2e824ef0a"
-          (reference "R9") (unit 1)
-        )
-        (path "/c83c6236-96e9-46ad-9d7a-9e2efa4a7966/5fc618b8-7830-4bbf-bf46-7753631e9b1e"
-          (reference "R11") (unit 1)
-        )
-        (path "/c83c6236-96e9-46ad-9d7a-9e2efa4a7966/f06c9bf0-de4e-49a2-91ec-1c9426377826"
-          (reference "R19") (unit 1)
-        )
-        (path "/c83c6236-96e9-46ad-9d7a-9e2efa4a7966/803edf1a-5825-4947-a8b9-85d3a29697e5"
-          (reference "R15") (unit 1)
-        )
         (path "/c83c6236-96e9-46ad-9d7a-9e2efa4a7966/802175d5-fb4b-4457-a117-b0f397189ff7"
           (reference "R13") (unit 1)
-        )
-        (path "/c83c6236-96e9-46ad-9d7a-9e2efa4a7966/ef548cdc-9d5d-4f8e-8f54-0c2e96dbe3f0"
-          (reference "R1") (unit 1)
         )
         (path "/c83c6236-96e9-46ad-9d7a-9e2efa4a7966/c9e1b2da-9064-45a5-a0a2-ee072f7e1acf"
@@
     )
   )
-  (symbol (lib_id "power:GNDD") (at 116.84 130.81 0) (unit 1)
-    (in_bom yes) (on_board yes) (dnp no) (fields_autoplaced)
-    (property "Reference" "#PWR071" (at 116.84 137.16 0)
-      (effects (font (size 1.27 1.27)) hide)
-    )
-    (property "Value" "GNDD" (at 116.84 134.62 0)
+  (symbol (lib_id "power:GNDD") (at 116.84 132.08 0) (unit 1)
+    (in_bom yes) (on_board yes) (dnp no) (fields_autoplaced)
+    (property "Reference" "#PWR071" (at 116.84 138.43 0)
+      (effects (font (size 1.27 1.27)) hide)
+    )
+    (property "Value" "GNDD" (at 116.84 135.89 0)
       (effects (font (size 1.27 1.27)))
     )
-    (property "Footprint" "" (at 116.84 130.81 0)
-      (effects (font (size 1.27 1.27)) hide)
-    )
-    (property "Datasheet" "" (at 116.84 130.81 0)
-      (effects (font (size 1.27 1.27)) hide)
-    )
+    (property "Footprint" "" (at 116.84 132.08 0)
+      (effects (font (size 1.27 1.27)) hide)
+    )
+    (property "Datasheet" "" (at 116.84 132.08 0)
+      (effects (font (size 1.27 1.27)) hide)
+    )

Commit message: reannotated and did some more cleanup.  almost ready
Parts:
- renumbered R1 to R13, U6 to U4
Other:
- company: (none) -> github.com/hoeken/yarrboard
- title: (none) -> RGB Input Board
Changed lines of the file:
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@@
 (kicad_sch (version 20230121) (generator eeschema)
   (paper "A4")
+  (title_block
+    (title "RGB Input Board")
+    (rev "B")
+    (company "github.com/hoeken/yarrboard")
+    (comment 1 "Open Source Hardware")
+  )
   (junction (at 121.92 52.07) (diameter 0) (color 0 0 0 0)
   )
@@
   (symbol (lib_id "power:GNDD") (at 72.39 78.74 0) (unit 1)
     (in_bom yes) (on_board yes) (dnp no) (fields_autoplaced)
-    (property "Reference" "#PWR073" (at 72.39 85.09 0)
+    (property "Reference" "#PWR053" (at 72.39 85.09 0)
       (effects (font (size 1.27 1.27)) hide)
     )
@@
       (project "rgb-input"
         (path "/c83c6236-96e9-46ad-9d7a-9e2efa4a7966/846833bc-7ec6-4ec6-86e7-310fef01b65c/720a8c4a-525c-4eec-8216-6ac4d044fce4"
-          (reference "#PWR073") (unit 1)
+          (reference "#PWR053") (unit 1)
         )
       )
@@
   (symbol (lib_id "Device:R_US") (at 95.25 80.01 0) (mirror x) (unit 1)
     (in_bom yes) (on_board yes) (dnp no) (fields_autoplaced)
-    (property "Reference" "R1" (at 92.71 78.74 0)
+    (property "Reference" "R13" (at 92.71 78.74 0)
       (effects (font (size 1.27 1.27)) (justify right))
     )
@@
     (instances
       (project "rgb-input"
+        (path "/c83c6236-96e9-46ad-9d7a-9e2efa4a7966/802175d5-fb4b-4457-a117-b0f397189ff7"
+          (reference "R13") (unit 1)
+        )
+        (path "/c83c6236-96e9-46ad-9d7a-9e2efa4a7966/4f50afed-9381-4977-8e27-209f0f88ad4e"
+          (reference "R3") (unit 1)
+        )
+        (path "/c83c6236-96e9-46ad-9d7a-9e2efa4a7966/4175a172-5c0b-4d6a-88bb-129f5f07b813"
+          (reference "R5") (unit 1)
+        )
+        (path "/c83c6236-96e9-46ad-9d7a-9e2efa4a7966/6f6f2d8d-82f6-4691-bba7-8caa1bd52e96"
+          (reference "R7") (unit 1)
+        )
+        (path "/c83c6236-96e9-46ad-9d7a-9e2efa4a7966/145fa34f-e19e-43e2-bb48-aff2e824ef0a"
+          (reference "R9") (unit 1)
+        )
+        (path "/c83c6236-96e9-46ad-9d7a-9e2efa4a7966/5fc618b8-7830-4bbf-bf46-7753631e9b1e"
+          (reference "R11") (unit 1)
+        )
+        (path "/c83c6236-96e9-46ad-9d7a-9e2efa4a7966/f06c9bf0-de4e-49a2-91ec-1c9426377826"
+          (reference "R19") (unit 1)
+        )
+        (path "/c83c6236-96e9-46ad-9d7a-9e2efa4a7966/803edf1a-5825-4947-a8b9-85d3a29697e5"
+          (reference "R15") (unit 1)
+        )
         (path "/c83c6236-96e9-46ad-9d7a-9e2efa4a7966/ef548cdc-9d5d-4f8e-8f54-0c2e96dbe3f0"
           (reference "R1") (unit 1)
         )
-        (path "/c83c6236-96e9-46ad-9d7a-9e2efa4a7966/4f50afed-9381-4977-8e27-209f0f88ad4e"
-          (reference "R3") (unit 1)
-        )
-        (path "/c83c6236-96e9-46ad-9d7a-9e2efa4a7966/4175a172-5c0b-4d6a-88bb-129f5f07b813"
-          (reference "R5") (unit 1)
-        )
-        (path "/c83c6236-96e9-46ad-9d7a-9e2efa4a7966/6f6f2d8d-82f6-4691-bba7-8caa1bd52e96"
-          (reference "R7") (unit 1)
-        )
-        (path "/c83c6236-96e9-46ad-9d7a-9e2efa4a7966/145fa34f-e19e-43e2-bb48-aff2e824ef0a"
-          (reference "R9") (unit 1)
-        )
-        (path "/c83c6236-96e9-46ad-9d7a-9e2efa4a7966/5fc618b8-7830-4bbf-bf46-7753631e9b1e"
-          (reference "R11") (unit 1)
-        )
-        (path "/c83c6236-96e9-46ad-9d7a-9e2efa4a7966/f06c9bf0-de4e-49a2-91ec-1c9426377826"
-          (reference "R19") (unit 1)
-        )
-        (path "/c83c6236-96e9-46ad-9d7a-9e2efa4a7966/803edf1a-5825-4947-a8b9-85d3a29697e5"
-          (reference "R15") (unit 1)
-        )
         (path "/c83c6236-96e9-46ad-9d7a-9e2efa4a7966/120468c6-3bec-414c-9049-57af589f397a"
           (reference "R20") (unit 1)
         )
-        (path "/c83c6236-96e9-46ad-9d7a-9e2efa4a7966/802175d5-fb4b-4457-a117-b0f397189ff7"
-          (reference "R13") (unit 1)
-        )
         (path "/c83c6236-96e9-46ad-9d7a-9e2efa4a7966/c9e1b2da-9064-45a5-a0a2-ee072f7e1acf"
           (reference "R21") (unit 1)
@@
         )
         (path "/c83c6236-96e9-46ad-9d7a-9e2efa4a7966/846833bc-7ec6-4ec6-86e7-310fef01b65c/720a8c4a-525c-4eec-8216-6ac4d044fce4"
-          (reference "R48") (unit 1)
+          (reference "R30") (unit 1)
         )
       )
@@
   (symbol (lib_id "power:+3.3V") (at 121.92 50.8 0) (unit 1)
     (in_bom yes) (on_board yes) (dnp no) (fields_autoplaced)
-    (property "Reference" "#PWR082" (at 121.92 54.61 0)
+    (property "Reference" "#PWR052" (at 121.92 54.61 0)
       (effects (font (size 1.27 1.27)) hide)
     )
@@
       (project "rgb-input"
         (path "/c83c6236-96e9-46ad-9d7a-9e2efa4a7966/846833bc-7ec6-4ec6-86e7-310fef01b65c/720a8c4a-525c-4eec-8216-6ac4d044fce4"
-          (reference "#PWR082") (unit 1)
+          (reference "#PWR052") (unit 1)
         )
       )
@@
         )
         (path "/c83c6236-96e9-46ad-9d7a-9e2efa4a7966/846833bc-7ec6-4ec6-86e7-310fef01b65c/720a8c4a-525c-4eec-8216-6ac4d044fce4"
-          (reference "C26") (unit 1)
+          (reference "C23") (unit 1)
         )
       )
@@
   (symbol (lib_id "power:GNDD") (at 116.84 132.08 0) (unit 1)
     (in_bom yes) (on_board yes) (dnp no) (fields_autoplaced)
-    (property "Reference" "#PWR071" (at 116.84 138.43 0)
+    (property "Reference" "#PWR054" (at 116.84 138.43 0)
       (effects (font (size 1.27 1.27)) hide)
     )
@@
       (project "rgb-input"
         (path "/c83c6236-96e9-46ad-9d7a-9e2efa4a7966/846833bc-7ec6-4ec6-86e7-310fef01b65c/720a8c4a-525c-4eec-8216-6ac4d044fce4"
-          (reference "#PWR071") (unit 1)
+          (reference "#PWR054") (unit 1)
         )
       )
@@
   (symbol (lib_id "Driver_LED:TLC5947DAP") (at 116.84 91.44 0) (unit 1)
     (in_bom yes) (on_board yes) (dnp no)
-    (property "Reference" "U6" (at 102.87 53.34 0)
+    (property "Reference" "U4" (at 102.87 53.34 0)
       (effects (font (size 1.27 1.27)) (justify left))
     )
@@
       (project "rgb-input"
         (path "/c83c6236-96e9-46ad-9d7a-9e2efa4a7966/846833bc-7ec6-4ec6-86e7-310fef01b65c/720a8c4a-525c-4eec-8216-6ac4d044fce4"
-          (reference "U6") (unit 1)
-        )
-      )
+          (reference "U4") (unit 1)
+        )
+      )
