File: boards/rgb-input/leds.kicad_sch (KiCad schematic)
At the start: 1 part, among them J46 RGB

Commit message: new rgb input board coming along very nicely
Parts:
- J46: footprint Connector_IDC:IDC-Header_2x25_P2.54mm_Vertical -> Connector_FFC-FPC:Molex_200528-0300_1x30-1MP_P1.00mm_Horizontal; symbol Connector_Generic:Conn_02x25_Odd_Even -> Connector_Generic:Conn_01x30
Connections:
- net +5V: now also J46.2 (Pin_2), J46.3 (Pin_3)
- net BLUE0: now also J46.9 (Pin_9); no longer J46.12 (Pin_12)
- net BLUE1: now also J46.12 (Pin_12); no longer J46.9 (Pin_9)
- net BLUE2: now also J46.15 (Pin_15); no longer J46.6 (Pin_6)
- net BLUE3: now also J46.18 (Pin_18); no longer J46.3 (Pin_3)
- net BLUE4: now also J46.21 (Pin_21); no longer J46.17 (Pin_17)
- net BLUE5: now also J46.24 (Pin_24); no longer J46.20 (Pin_20)
- net BLUE6: now also J46.27 (Pin_27); no longer J46.23 (Pin_23)
- net BLUE7: now also J46.30 (Pin_30); no longer J46.26 (Pin_26)
- net GNDD: now also J46.4 (Pin_4), J46.5 (Pin_5), J46.6 (Pin_6); no longer J46.2 (Pin_2)
- net GREEN0: now also J46.8 (Pin_8); no longer J46.13 (Pin_13)
- net GREEN1: now also J46.11 (Pin_11); no longer J46.10 (Pin_10)
- net GREEN2: now also J46.14 (Pin_14); no longer J46.7 (Pin_7)
- net GREEN3: now also J46.17 (Pin_17); no longer J46.4 (Pin_4)
- net GREEN4: now also J46.20 (Pin_20); no longer J46.16 (Pin_16)
- net GREEN5: now also J46.23 (Pin_23); no longer J46.19 (Pin_19)
- net GREEN6: now also J46.26 (Pin_26); no longer J46.22 (Pin_22)
- net GREEN7: now also J46.29 (Pin_29); no longer J46.25 (Pin_25)
- net RED0: now also J46.7 (Pin_7); no longer J46.14 (Pin_14)
- net RED1: now also J46.10 (Pin_10); no longer J46.11 (Pin_11)
- net RED2: now also J46.13 (Pin_13); no longer J46.8 (Pin_8)
- net RED3: now also J46.16 (Pin_16); no longer J46.5 (Pin_5)
- net RED4: now also J46.19 (Pin_19); no longer J46.15 (Pin_15)
- net RED5: now also J46.22 (Pin_22); no longer J46.18 (Pin_18)
- net RED6: now also J46.25 (Pin_25); no longer J46.21 (Pin_21)
- net RED7: now also J46.28 (Pin_28); no longer J46.24 (Pin_24)

Commit message: new rgb input board is starting to look very nice.
Parts:
- J46: footprint Connector_FFC-FPC:Molex_200528-0300_1x30-1MP_P1.00mm_Horizontal -> Connector_FFC-FPC:TE_3-84952-0_1x30-1MP_P1.0mm_Horizontal
Changed lines of the file:
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@@
       (effects (font (size 1.27 1.27)) (justify left))
     )
-    (property "Footprint" "Connector_FFC-FPC:Molex_200528-0300_1x30-1MP_P1.00mm_Horizontal" (at 213.36 88.9 0)
+    (property "Footprint" "Connector_FFC-FPC:TE_3-84952-0_1x30-1MP_P1.0mm_Horizontal" (at 213.36 88.9 0)
       (effects (font (size 1.27 1.27)) hide)
     )

Commit message: passing ERC and DRC
Parts:
- J46: symbol Connector_Generic:Conn_01x30 -> Connector_Generic_MountingPin:Conn_01x30_MountingPin
Connections:
- net GNDD: now also J46.MP (MountPin)

Commit message: reannotated and did some more cleanup.  almost ready
Parts:
- renumbered J46 to J4
Other:
- company: (none) -> github.com/hoeken/yarrboard
- title: (none) -> RGB Input Board
Changed lines of the file:
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@@
 (kicad_sch (version 20230121) (generator eeschema)
   (paper "A4")
+  (title_block
+    (title "RGB Input Board")
+    (rev "B")
+    (company "github.com/hoeken/yarrboard")
+    (comment 1 "Open Source Hardware")
+  )
   (junction (at 195.58 66.04) (diameter 0) (color 0 0 0 0)
   )
@@
   (symbol (lib_id "power:+5V") (at 195.58 50.8 0) (unit 1)
     (in_bom yes) (on_board yes) (dnp no) (fields_autoplaced)
-    (property "Reference" "#PWR098" (at 195.58 54.61 0)
+    (property "Reference" "#PWR060" (at 195.58 54.61 0)
       (effects (font (size 1.27 1.27)) hide)
     )
@@
       (project "rgb-input"
         (path "/c83c6236-96e9-46ad-9d7a-9e2efa4a7966/846833bc-7ec6-4ec6-86e7-310fef01b65c"
-          (reference "#PWR098") (unit 1)
+          (reference "#PWR060") (unit 1)
         )
       )
@@
         )
         (path "/c83c6236-96e9-46ad-9d7a-9e2efa4a7966/846833bc-7ec6-4ec6-86e7-310fef01b65c"
-          (reference "#PWR039") (unit 1)
+          (reference "#PWR062") (unit 1)
         )
       )
@@
         )
         (path "/c83c6236-96e9-46ad-9d7a-9e2efa4a7966/846833bc-7ec6-4ec6-86e7-310fef01b65c"
-          (reference "#PWR099") (unit 1)
+          (reference "#PWR061") (unit 1)
         )
       )
@@
   (symbol (lib_id "Connector_Generic_MountingPin:Conn_01x30_MountingPin") (at 213.36 88.9 0) (unit 1)
     (in_bom yes) (on_board yes) (dnp no) (fields_autoplaced)
-    (property "Reference" "J46" (at 215.9 89.2556 0)
+    (property "Reference" "J4" (at 215.9 89.2556 0)
       (effects (font (size 1.27 1.27)) (justify left))
     )
@@
       (project "rgb-input"
         (path "/c83c6236-96e9-46ad-9d7a-9e2efa4a7966/846833bc-7ec6-4ec6-86e7-310fef01b65c"
-          (reference "J46") (unit 1)
+          (reference "J4") (unit 1)
         )
       )

Commit message: parts list updated
Parts:
- J4: LCSC C30006 -> C262358; Manufacturer (none) -> AFA07-S30FCC-00
Changed lines of the file:
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@@
       (effects (font (size 1.27 1.27)) hide)
     )
-    (property "LCSC" "C30006" (at 213.36 88.9 0)
+    (property "LCSC" "C262358" (at 213.36 88.9 0)
       (effects (font (size 1.27 1.27)) hide)
     )
+    (property "Manufacturer" "AFA07-S30FCC-00" (at 213.36 88.9 0)
+      (effects (font (size 1.27 1.27)) hide)
+    )
